File: hardware/kicad/module-tile/counter.kicad_sch (KiCad schematic)
At the start: 3 parts, among them U3 74LS161, U3 74LS73, U4 74AUC2G08

Commit message: Schematics update
Parts:
- renumbered U3 to U1, U4 to U2
Changed lines of the file:
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@@
 		(on_board yes)
 		(dnp no)
-		(property "Reference" "U3"
+		(property "Reference" "U1"
 			(at 83.82 107.95 0)
 			(effects
@@
 		(instances
 			(project "tastiera_isomorfa"
-				(path "/2a6329ec-b0e8-4012-8f5a-476608b8b2cc/b0937e1a-84b9-4c23-9b14-d9868eedff6e"
-					(reference "U3")
+				(path "/2a6329ec-b0e8-4012-8f5a-476608b8b2cc/07e251ec-a89a-41e0-b307-1d6ec78f24c5/41fc8254-caa5-4a09-ad79-5b9ed9e5d35c"
+					(reference "U1")
 					(unit 1)
 				)
@@
 		(dnp no)
 		(fields_autoplaced yes)
-		(property "Reference" "#PWR07"
+		(property "Reference" "#PWR01"
 			(at 95.25 125.73 0)
 			(effects
@@
 		(instances
 			(project "tastiera_isomorfa"
-				(path "/2a6329ec-b0e8-4012-8f5a-476608b8b2cc/b0937e1a-84b9-4c23-9b14-d9868eedff6e"
-					(reference "#PWR07")
+				(path "/2a6329ec-b0e8-4012-8f5a-476608b8b2cc/07e251ec-a89a-41e0-b307-1d6ec78f24c5/41fc8254-caa5-4a09-ad79-5b9ed9e5d35c"
+					(reference "#PWR01")
 					(unit 1)
 				)
@@
 		(dnp no)
 		(fields_autoplaced yes)
-		(property "Reference" "#PWR05"
+		(property "Reference" "#PWR04"
 			(at 187.96 154.94 0)
 			(effects
@@
 		(instances
 			(project "tastiera_isomorfa"
-				(path "/2a6329ec-b0e8-4012-8f5a-476608b8b2cc/b0937e1a-84b9-4c23-9b14-d9868eedff6e"
-					(reference "#PWR05")
+				(path "/2a6329ec-b0e8-4012-8f5a-476608b8b2cc/07e251ec-a89a-41e0-b307-1d6ec78f24c5/41fc8254-caa5-4a09-ad79-5b9ed9e5d35c"
+					(reference "#PWR04")
 					(unit 1)
 				)
@@
 		(dnp no)
 		(fields_autoplaced yes)
-		(property "Reference" "U4"
+		(property "Reference" "U2"
 			(at 124.4711 90.17 0)
 			(effects
@@
 		(instances
 			(project "tastiera_isomorfa"
-				(path "/2a6329ec-b0e8-4012-8f5a-476608b8b2cc/b0937e1a-84b9-4c23-9b14-d9868eedff6e"
-					(reference "U4")
+				(path "/2a6329ec-b0e8-4012-8f5a-476608b8b2cc/07e251ec-a89a-41e0-b307-1d6ec78f24c5/41fc8254-caa5-4a09-ad79-5b9ed9e5d35c"
+					(reference "U2")
 					(unit 1)
 				)
@@
 		(dnp no)
 		(fields_autoplaced yes)
-		(property "Reference" "#PWR03"
+		(property "Reference" "#PWR05"
 			(at 193.04 82.55 0)
 			(effects
@@
 		(instances
 			(project "tastiera_isomorfa"
-				(path "/2a6329ec-b0e8-4012-8f5a-476608b8b2cc/b0937e1a-84b9-4c23-9b14-d9868eedff6e"
-					(reference "#PWR03")
+				(path "/2a6329ec-b0e8-4012-8f5a-476608b8b2cc/07e251ec-a89a-41e0-b307-1d6ec78f24c5/41fc8254-caa5-4a09-ad79-5b9ed9e5d35c"
+					(reference "#PWR05")
 					(unit 1)
 				)
@@
 		(instances
 			(project "tastiera_isomorfa"
-				(path "/2a6329ec-b0e8-4012-8f5a-476608b8b2cc/b0937e1a-84b9-4c23-9b14-d9868eedff6e"
+				(path "/2a6329ec-b0e8-4012-8f5a-476608b8b2cc/07e251ec-a89a-41e0-b307-1d6ec78f24c5/41fc8254-caa5-4a09-ad79-5b9ed9e5d35c"
 					(reference "U3")
 					(unit 1)
@@
 		(dnp no)
 		(fields_autoplaced yes)
-		(property "Reference" "#PWR06"
+		(property "Reference" "#PWR03"
 			(at 162.56 154.94 0)
 			(effects
@@
 		(instances
 			(project "tastiera_isomorfa"
-				(path "/2a6329ec-b0e8-4012-8f5a-476608b8b2cc/b0937e1a-84b9-4c23-9b14-d9868eedff6e"
-					(reference "#PWR06")
+				(path "/2a6329ec-b0e8-4012-8f5a-476608b8b2cc/07e251ec-a89a-41e0-b307-1d6ec78f24c5/41fc8254-caa5-4a09-ad79-5b9ed9e5d35c"
+					(reference "#PWR03")
 					(unit 1)
 				)
@@
 		(dnp no)
 		(fields_autoplaced yes)
-		(property "Reference" "#PWR04"
+		(property "Reference" "#PWR02"
 			(at 162.56 82.55 0)
 			(effects
@@
 		(instances
 			(project "tastiera_isomorfa"
-				(path "/2a6329ec-b0e8-4012-8f5a-476608b8b2cc/b0937e1a-84b9-4c23-9b14-d9868eedff6e"
-					(reference "#PWR04")
-					(unit 1)
-				)
+				(path "/2a6329ec-b0e8-4012-8f5a-476608b8b2cc/07e251ec-a89a-41e0-b307-1d6ec78f24c5/41fc8254-caa5-4a09-ad79-5b9ed9e5d35c"
+					(reference "#PWR02")
+					(unit 1)
+				)

Commit message: Schematic complete
Parts:
- removed U1: 74LS73, symbol 74xx:74LS73
- added U106: 74LVC2G32, Package_SO:MSOP-8_3x3mm_P0.65mm, symbol 74xGxx:74LVC2G32
- added U108: 74LVC2G74, Package_SO:MSOP-8_3x3mm_P0.65mm, symbol 74xGxx:74LVC2G74
- U102: renamed from U2; footprint (none) -> Package_SO:MSOP-8_3x3mm_P0.65mm; Codice (none) -> SN74LVC2G08IDCTRQ1; Link (none) -> https://www.digikey.it/it/products/detail/texas-instruments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
- U109: renamed from U3; footprint (none) -> Package_SO:SOIC-16_3.9x9.9mm_P1.27mm; Codice (none) -> SN74HC161DR; Link (none) -> https://www.digikey.it/it/products/detail/texas-instruments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
Connections:
- net GND: now also U108.4 (GND)
- net Q: now also U106.5, U108.5 (Q)
- net VCC: now also U108.7 (~{PRE}), U108.8 (VCC)
- net clk: now also U108.1 (C)
- net ~{rst}: now also U108.6 (~{CLR})
- net at U102.7: now also U106.6
- new net: U106.3, U108.2 (D)
Other:
- moved on the sheet: U102A, U109
