File: hardware/kicad/module-tile/keyboard.kicad_sch (KiCad schematic)
At the start: 12 parts, among them SW1 SW_Push, SW10 SW_Push, SW11 SW_Push, SW12 SW_Push, SW2 SW_Push, SW3 SW_Push, SW4 SW_Push, SW5 SW_Push, SW6 SW_Push, SW7 SW_Push, SW8 SW_Push, SW9 SW_Push

Commit message: Improving schematics
Parts:
- added R1, R10, R11, R12, R2, R3, R4, R5, R6, R7, R8, R9: 10k, symbol Device:R
- added R13, R14, R15, R16, R17, R18, R19, R20, R21, R22, R23, R24: 100R, symbol Device:R
Connections:
- net BTNs0: now also R13.2; no longer SW1.2
- net BTNs1: now also R14.2; no longer SW2.2
- net BTNs10: now also R23.2; no longer SW11.2
- net BTNs11: now also R24.2; no longer SW12.2
- net BTNs2: now also R15.2; no longer SW3.2
- net BTNs3: now also R16.2; no longer SW4.2
- net BTNs4: now also R17.2; no longer SW5.2
- net BTNs5: now also R18.2; no longer SW6.2
- net BTNs6: now also R19.2; no longer SW7.2
- net BTNs7: now also R20.2; no longer SW8.2
- net BTNs8: now also R21.2; no longer SW9.2
- net BTNs9: now also R22.2; no longer SW10.2
- net VCC: now reaches SW1.1, SW10.1, SW11.1, SW12.1, SW2.1, SW3.1, SW4.1, SW5.1, SW6.1, SW7.1, SW8.1, SW9.1
- new net: R1.1, R13.1, SW1.2
- new net: R12.1, R24.1, SW12.2
- new net: R16.1, R4.1, SW4.2
- new net: R15.1, R3.1, SW3.2
- new net: R21.1, R9.1, SW9.2
- new net: R11.1, R23.1, SW11.2
- new net: R10.1, R22.1, SW10.2
- new net: R20.1, R8.1, SW8.2
- new net: R18.1, R6.1, SW6.2
- new net: R17.1, R5.1, SW5.2
- new net: R14.1, R2.1, SW2.2
- new net: R19.1, R7.1, SW7.2
- new net GND: R1.2, R10.2, R11.2, R12.2, R2.2, R3.2, R4.2, R5.2, R6.2, R7.2, R8.2, R9.2
Other:
- moved on the sheet: SW1, SW10, SW11, SW12, SW2, SW3, SW4, SW5, SW6, SW7, SW8, SW9

Commit message: Schematics update
Parts:
- renumbered R13 to R1, R22 to R10, R23 to R11, R24 to R12, R1 to R13, R2 to R14, R3 to R15, R4 to R16, R5 to R17, R6 to R18, R7 to R19, R14 to R2, R8 to R20, R9 to R21, R10 to R22, R11 to R23, R12 to R24, R15 to R3, R16 to R4, R17 to R5, R18 to R6, R19 to R7, R20 to R8, R21 to R9

Commit message: Schematic complete
Parts:
- R110: renamed from R1; footprint (none) -> Resistor_SMD:R_0805_2012Metric_Pad1.20x1.40mm_HandSolder; Codice (none) -> CRCW0805100RFKEA; Link (none) -> https://www.digikey.it/it/products/detail/vishay-dale/CRCW0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
- R111: renamed from R2; footprint (none) -> Resistor_SMD:R_0805_2012Metric_Pad1.20x1.40mm_HandSolder; Codice (none) -> CRCW0805100RFKEA; Link (none) -> https://www.digikey.it/it/products/detail/vishay-dale/CRCW0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
- R112: renamed from R3; footprint (none) -> Resistor_SMD:R_0805_2012Metric_Pad1.20x1.40mm_HandSolder; Codice (none) -> CRCW0805100RFKEA; Link (none) -> https://www.digikey.it/it/products/detail/vishay-dale/CRCW0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
- R113: renamed from R4; footprint (none) -> Resistor_SMD:R_0805_2012Metric_Pad1.20x1.40mm_HandSolder; Codice (none) -> CRCW0805100RFKEA; Link (none) -> https://www.digikey.it/it/products/detail/vishay-dale/CRCW0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
- R114: renamed from R5; footprint (none) -> Resistor_SMD:R_0805_2012Metric_Pad1.20x1.40mm_HandSolder; Codice (none) -> CRCW0805100RFKEA; Link (none) -> https://www.digikey.it/it/products/detail/vishay-dale/CRCW0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
- R115: renamed from R6; footprint (none) -> Resistor_SMD:R_0805_2012Metric_Pad1.20x1.40mm_HandSolder; Codice (none) -> CRCW0805100RFKEA; Link (none) -> https://www.digikey.it/it/products/detail/vishay-dale/CRCW0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
- R116: renamed from R7; footprint (none) -> Resistor_SMD:R_0805_2012Metric_Pad1.20x1.40mm_HandSolder; Codice (none) -> CRCW0805100RFKEA; Link (none) -> https://www.digikey.it/it/products/detail/vishay-dale/CRCW0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
- R117: renamed from R8; footprint (none) -> Resistor_SMD:R_0805_2012Metric_Pad1.20x1.40mm_HandSolder; Codice (none) -> CRCW0805100RFKEA; Link (none) -> https://www.digikey.it/it/products/detail/vishay-dale/CRCW0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
- R118: renamed from R9; footprint (none) -> Resistor_SMD:R_0805_2012Metric_Pad1.20x1.40mm_HandSolder; Codice (none) -> CRCW0805100RFKEA; Link (none) -> https://www.digikey.it/it/products/detail/vishay-dale/CRCW0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
- R119: renamed from R10; footprint (none) -> Resistor_SMD:R_0805_2012Metric_Pad1.20x1.40mm_HandSolder; Codice (none) -> CRCW0805100RFKEA; Link (none) -> https://www.digikey.it/it/products/detail/vishay-dale/CRCW0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
- R120: renamed from R11; footprint (none) -> Resistor_SMD:R_0805_2012Metric_Pad1.20x1.40mm_HandSolder; Codice (none) -> CRCW0805100RFKEA; Link (none) -> https://www.digikey.it/it/products/detail/vishay-dale/CRCW0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
- R121: renamed from R12; footprint (none) -> Resistor_SMD:R_0805_2012Metric_Pad1.20x1.40mm_HandSolder; Codice (none) -> CRCW0805100RFKEA; Link (none) -> https://www.digikey.it/it/products/detail/vishay-dale/CRCW0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
- R122: renamed from R13; footprint (none) -> Resistor_SMD:R_0805_2012Metric_Pad1.20x1.40mm_HandSolder; Codice (none) -> RMCF0805FT10K0; Link (none) -> https://www.digikey.it/it/products/detail/stackpole-electro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
- R123: renamed from R14; footprint (none) -> Resistor_SMD:R_0805_2012Metric_Pad1.20x1.40mm_HandSolder; Codice (none) -> RMCF0805FT10K0; Link (none) -> https://www.digikey.it/it/products/detail/stackpole-electro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
- R124: renamed from R15; footprint (none) -> Resistor_SMD:R_0805_2012Metric_Pad1.20x1.40mm_HandSolder; Codice (none) -> RMCF0805FT10K0; Link (none) -> https://www.digikey.it/it/products/detail/stackpole-electro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
- R125: renamed from R16; footprint (none) -> Resistor_SMD:R_0805_2012Metric_Pad1.20x1.40mm_HandSolder; Codice (none) -> RMCF0805FT10K0; Link (none) -> https://www.digikey.it/it/products/detail/stackpole-electro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
- R126: renamed from R17; footprint (none) -> Resistor_SMD:R_0805_2012Metric_Pad1.20x1.40mm_HandSolder; Codice (none) -> RMCF0805FT10K0; Link (none) -> https://www.digikey.it/it/products/detail/stackpole-electro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
- R127: renamed from R18; footprint (none) -> Resistor_SMD:R_0805_2012Metric_Pad1.20x1.40mm_HandSolder; Codice (none) -> RMCF0805FT10K0; Link (none) -> https://www.digikey.it/it/products/detail/stackpole-electro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
- R128: renamed from R19; footprint (none) -> Resistor_SMD:R_0805_2012Metric_Pad1.20x1.40mm_HandSolder; Codice (none) -> RMCF0805FT10K0; Link (none) -> https://www.digikey.it/it/products/detail/stackpole-electro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
- R129: renamed from R20; footprint (none) -> Resistor_SMD:R_0805_2012Metric_Pad1.20x1.40mm_HandSolder; Codice (none) -> RMCF0805FT10K0; Link (none) -> https://www.digikey.it/it/products/detail/stackpole-electro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
- R130: renamed from R21; footprint (none) -> Resistor_SMD:R_0805_2012Metric_Pad1.20x1.40mm_HandSolder; Codice (none) -> RMCF0805FT10K0; Link (none) -> https://www.digikey.it/it/products/detail/stackpole-electro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
- R131: renamed from R22; footprint (none) -> Resistor_SMD:R_0805_2012Metric_Pad1.20x1.40mm_HandSolder; Codice (none) -> RMCF0805FT10K0; Link (none) -> https://www.digikey.it/it/products/detail/stackpole-electro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
- R132: renamed from R23; footprint (none) -> Resistor_SMD:R_0805_2012Metric_Pad1.20x1.40mm_HandSolder; Codice (none) -> RMCF0805FT10K0; Link (none) -> https://www.digikey.it/it/products/detail/stackpole-electro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
- R133: renamed from R24; footprint (none) -> Resistor_SMD:R_0805_2012Metric_Pad1.20x1.40mm_HandSolder; Codice (none) -> RMCF0805FT10K0; Link (none) -> https://www.digikey.it/it/products/detail/stackpole-electro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
- SW101: renamed from SW1; footprint (none) -> Button_Switch_Keyboard:SW_Cherry_MX_1.00u_PCB
- SW102: renamed from SW2; footprint (none) -> Button_Switch_Keyboard:SW_Cherry_MX_1.00u_PCB
- SW103: renamed from SW3; footprint (none) -> Button_Switch_Keyboard:SW_Cherry_MX_1.00u_PCB
- SW104: renamed from SW4; footprint (none) -> Button_Switch_Keyboard:SW_Cherry_MX_1.00u_PCB
- SW105: renamed from SW5; footprint (none) -> Button_Switch_Keyboard:SW_Cherry_MX_1.00u_PCB
- SW106: renamed from SW6; footprint (none) -> Button_Switch_Keyboard:SW_Cherry_MX_1.00u_PCB
- SW107: renamed from SW7; footprint (none) -> Button_Switch_Keyboard:SW_Cherry_MX_1.00u_PCB
- SW108: renamed from SW8; footprint (none) -> Button_Switch_Keyboard:SW_Cherry_MX_1.00u_PCB
- SW109: renamed from SW9; footprint (none) -> Button_Switch_Keyboard:SW_Cherry_MX_1.00u_PCB
- SW110: renamed from SW10; footprint (none) -> Button_Switch_Keyboard:SW_Cherry_MX_1.00u_PCB
- SW111: renamed from SW11; footprint (none) -> Button_Switch_Keyboard:SW_Cherry_MX_1.00u_PCB
- SW112: renamed from SW12; footprint (none) -> Button_Switch_Keyboard:SW_Cherry_MX_1.00u_PCB

Commit message: Pcb started
Changed lines of the file:
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@@
+		)
+	)
+	(bus
+		(pts
+			(xy 161.29 39.37) (xy 161.29 49.53)
+		)
+		(stroke
+			(width 0)
+			(type default)
 		)
 	)
@@
 		)
 	)
+	(wire
+		(pts
+			(xy 110.49 82.55) (xy 110.49 92.71)
+		)
+		(stroke
+			(width 0)
+			(type default)
+		)
+	)
+	(wire
+		(pts
+			(xy 135.89 62.23) (xy 138.43 62.23)
+		)
+		(stroke
+			(width 0)
+			(type default)
+		)
+	)
+	(wire
+		(pts
+			(xy 110.49 123.19) (xy 110.49 133.35)
+		)
+		(stroke
+			(width 0)
+			(type default)
+		)
+	)
+	(wire
+		(pts
+			(xy 120.65 153.67) (xy 110.49 153.67)
+		)
+		(stroke
+			(width 0)
+			(type default)
+		)
+	)
+	(wire
+		(pts
+			(xy 182.88 86.36) (xy 182.88 91.44)
+		)
+		(stroke
+			(width 0)
+			(type default)
+		)
+	)
+	(wire
+		(pts
+			(xy 195.58 96.52) (xy 195.58 91.44)
+		)
+		(stroke
+			(width 0)
+			(type default)
+		)
+	)
+	(wire
+		(pts
+			(xy 176.53 66.04) (xy 182.88 66.04)
+		)
+		(stroke
+			(width 0)
+			(type default)
+		)
+	)
+	(wire
+		(pts
+			(xy 130.81 153.67) (xy 135.89 153.67)
+		)
+		(stroke
+			(width 0)
+			(type default)
+		)
+	)
+	(wire
+		(pts
+			(xy 110.49 97.79) (xy 110.49 102.87)
+		)
+		(stroke
+			(width 0)
+			(type default)
+		)
+	)
 	(bus
 		(pts
+			(xy 161.29 69.85) (xy 161.29 80.01)
+		)
+		(stroke
+			(width 0)
+			(type default)
+		)
+	)
+	(wire
+		(pts
+			(xy 110.49 62.23) (xy 120.65 62.23)
+		)
+		(stroke
+			(width 0)
+			(type default)
+		)
+	)
+	(bus
+		(pts
 			(xy 161.29 33.02) (xy 161.29 39.37)
-		)
-		(stroke
-			(width 0)
-			(type default)
-		)
-	)
-	(wire
-		(pts
-			(xy 110.49 82.55) (xy 110.49 92.71)
-		)
-		(stroke
-			(width 0)
-			(type default)
-		)
-	)
-	(wire
-		(pts
-			(xy 135.89 62.23) (xy 138.43 62.23)
-		)
-		(stroke
-			(width 0)
-			(type default)
-		)
-	)
-	(wire
-		(pts
-			(xy 110.49 123.19) (xy 110.49 133.35)
-		)
-		(stroke
-			(width 0)
-			(type default)
-		)
-	)
-	(wire
-		(pts
-			(xy 120.65 153.67) (xy 110.49 153.67)
-		)
-		(stroke
-			(width 0)
-			(type default)
-		)
-	)
-	(wire
-		(pts
-			(xy 182.88 86.36) (xy 182.88 91.44)
-		)
-		(stroke
-			(width 0)
-			(type default)
-		)
-	)
-	(wire
-		(pts
-			(xy 195.58 96.52) (xy 195.58 91.44)
-		)
-		(stroke
-			(width 0)
-			(type default)
-		)
-	)
-	(wire
-		(pts
-			(xy 176.53 66.04) (xy 182.88 66.04)
-		)
-		(stroke
-			(width 0)
-			(type default)
-		)
-	)
-	(wire
-		(pts
-			(xy 130.81 153.67) (xy 135.89 153.67)
-		)
-		(stroke
-			(width 0)
-			(type default)
-		)
-	)
-	(wire
-		(pts
-			(xy 110.49 97.79) (xy 110.49 102.87)
-		)
-		(stroke
-			(width 0)
-			(type default)
-		)
-	)
-	(bus
-		(pts
-			(xy 161.29 69.85) (xy 161.29 80.01)
-		)
-		(stroke
-			(width 0)
-			(type default)
-		)
-	)
-	(wire
-		(pts
-			(xy 110.49 62.23) (xy 120.65 62.23)
-		)
-		(stroke
-			(width 0)
-			(type default)
-		)
-	)
-	(bus
-		(pts
-			(xy 161.29 39.37) (xy 161.29 49.53)
 		)
 		(stroke
@@
 		)
 	)
-	(hierarchical_label "BTNs"
+	(hierarchical_label "BTNs[0..11]"
 		(shape output)
 		(at 213.36 33.02 0)

Commit message: First commit new branch
Connections:
- net GND renamed GND_T
- net VCC renamed VCC_T
