File: hardware/kicad/module-tile/power.kicad_sch (KiCad schematic)
At the start: 9 parts, among them U1 74LS73, U2 74AUC2G08, U4 74AUC2G125, U5 74AUC2G126

Commit message: Schematic complete
Parts:
- removed C3, C4, C5: C, symbol Device:C
- removed U1: 74LS73, symbol 74xx:74LS73
- added C103, C104: 4u7, Capacitor_SMD:C_1206_3216Metric_Pad1.33x1.80mm_HandSolder, symbol Device:C_Polarized
- added C105: 100u, Capacitor_THT:CP_Radial_D6.3mm_P2.50mm, symbol Device:C_Polarized
- added U106: 74LVC2G32, Package_SO:MSOP-8_3x3mm_P0.65mm, symbol 74xGxx:74LVC2G32
- C101: renamed from C1; value C -> 100n; footprint (none) -> Capacitor_SMD:C_0805_2012Metric_Pad1.18x1.45mm_HandSolder; Codice (none) -> C0805C104K5RACTU; Link (none) -> https://www.digikey.it/it/products/detail/kemet/C0805C104K5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
- C102: renamed from C2; value C -> 100n; footprint (none) -> Capacitor_SMD:C_0805_2012Metric_Pad1.18x1.45mm_HandSolder; Codice (none) -> C0805C104K5RACTU; Link (none) -> https://www.digikey.it/it/products/detail/kemet/C0805C104K5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
- U101: renamed from U5; footprint (none) -> Package_SO:MSOP-8_3x3mm_P0.65mm; Codice (none) -> 74LVC2G126DCTRG4; Link (none) -> https://www.digikey.it/it/products/detail/texas-instruments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
- U102: renamed from U2; footprint (none) -> Package_SO:MSOP-8_3x3mm_P0.65mm; Codice (none) -> SN74LVC2G08IDCTRQ1; Link (none) -> https://www.digikey.it/it/products/detail/texas-instruments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
- U107: renamed from U4; footprint (none) -> Package_SO:MSOP-8_3x3mm_P0.65mm; Codice (none) -> SN74LVC2G125DCTR; Link (none) -> https://www.digikey.it/it/products/detail/texas-instruments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
Connections:
- net GND: now also C103.2, C104.2, C105.2, U106.4 (GND)
- net VCC: now also C103.1, C104.1, C105.1, U106.8 (VCC)
