File: hardware/kicad/module-tile/tile.kicad_sch (KiCad schematic)
At the start: 17 parts, among them U1 74HC165, U2 74HC165, U4 74AUC2G08, U5 74LS73, U6 74AUC2G125, U7 74AUC2G126, U8 74AHC1G32, U9 74AHC1G04

Commit message: Schematic complete
Parts:
- removed U5: 74LS73, symbol 74xx:74LS73
- removed U8: 74AHC1G32, symbol 74xGxx:74AHC1G32
- added U106: 74LVC2G32, Package_SO:MSOP-8_3x3mm_P0.65mm, symbol 74xGxx:74LVC2G32
- R101: renamed from R33; value R -> 10k; footprint (none) -> Resistor_SMD:R_0805_2012Metric_Pad1.20x1.40mm_HandSolder; Codice (none) -> RMCF0805FT10K0; Link (none) -> https://www.digikey.it/it/products/detail/stackpole-electro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
- R102: renamed from R29; value R -> 10k; footprint (none) -> Resistor_SMD:R_0805_2012Metric_Pad1.20x1.40mm_HandSolder; Codice (none) -> RMCF0805FT10K0; Link (none) -> https://www.digikey.it/it/products/detail/stackpole-electro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
- R103: renamed from R27; value R -> 10k; footprint (none) -> Resistor_SMD:R_0805_2012Metric_Pad1.20x1.40mm_HandSolder; Codice (none) -> RMCF0805FT10K0; Link (none) -> https://www.digikey.it/it/products/detail/stackpole-electro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
- R104: renamed from R25; value R -> 10k; footprint (none) -> Resistor_SMD:R_0805_2012Metric_Pad1.20x1.40mm_HandSolder; Codice (none) -> RMCF0805FT10K0; Link (none) -> https://www.digikey.it/it/products/detail/stackpole-electro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
- R105: renamed from R26; value R -> 10k; footprint (none) -> Resistor_SMD:R_0805_2012Metric_Pad1.20x1.40mm_HandSolder; Codice (none) -> RMCF0805FT10K0; Link (none) -> https://www.digikey.it/it/products/detail/stackpole-electro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
- R106: renamed from R32; value R -> 10k; footprint (none) -> Resistor_SMD:R_0805_2012Metric_Pad1.20x1.40mm_HandSolder; Codice (none) -> RMCF0805FT10K0; Link (none) -> https://www.digikey.it/it/products/detail/stackpole-electro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
- R107: renamed from R31; value R -> 10k; footprint (none) -> Resistor_SMD:R_0805_2012Metric_Pad1.20x1.40mm_HandSolder; Codice (none) -> RMCF0805FT10K0; Link (none) -> https://www.digikey.it/it/products/detail/stackpole-electro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
- R108: renamed from R30; value R -> 10k; footprint (none) -> Resistor_SMD:R_0805_2012Metric_Pad1.20x1.40mm_HandSolder; Codice (none) -> RMCF0805FT10K0; Link (none) -> https://www.digikey.it/it/products/detail/stackpole-electro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
- R109: renamed from R28; value R -> 10k; footprint (none) -> Resistor_SMD:R_0805_2012Metric_Pad1.20x1.40mm_HandSolder; Codice (none) -> RMCF0805FT10K0; Link (none) -> https://www.digikey.it/it/products/detail/stackpole-electro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
- U101: renamed from U7; footprint (none) -> Package_SO:MSOP-8_3x3mm_P0.65mm; Codice (none) -> 74LVC2G126DCTRG4; Link (none) -> https://www.digikey.it/it/products/detail/texas-instruments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
- U102: renamed from U4; footprint (none) -> Package_SO:MSOP-8_3x3mm_P0.65mm; Codice (none) -> SN74LVC2G08IDCTRQ1; Link (none) -> https://www.digikey.it/it/products/detail/texas-instruments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
- U103: renamed from U2; footprint (none) -> Package_SO:SOIC-16_3.9x9.9mm_P1.27mm; Codice (none) -> SN74LVC165ADR; Link (none) -> https://www.digikey.it/it/products/detail/texas-instruments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
- U104: renamed from U1; footprint (none) -> Package_SO:SOIC-16_3.9x9.9mm_P1.27mm; Codice (none) -> SN74LVC165ADR; Link (none) -> https://www.digikey.it/it/products/detail/texas-instruments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
- U105: renamed from U9; footprint (none) -> Package_TO_SOT_SMD:SOT-23-5_HandSoldering; Codice (none) -> SN74LVC1G04DBVR; Link (none) -> https://www.digikey.it/it/products/detail/texas-instruments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
- U107: renamed from U6; footprint (none) -> Package_SO:MSOP-8_3x3mm_P0.65mm; Codice (none) -> SN74LVC2G125DCTR; Link (none) -> https://www.digikey.it/it/products/detail/texas-instruments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
Connections:
- net B_latch: now also U106.1
- net L_latch: now also U106.7
- net R_latch: now also U106.2
- no-connect marks 8 -> 2

Commit message: Pcb started
Other:
- sheet keyboard ports: added BTNs[0..11]; removed BTNs
Changed lines of the file:
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@@
 	)
 	(junction
-		(at 191.77 151.13)
+		(at 199.39 73.66)
 		(diameter 0)
 		(color 0 0 0 0)
 	)
 	(junction
-		(at 228.6 146.05)
+		(at 191.77 151.13)
 		(diameter 0)
 		(color 0 0 0 0)
 	)
 	(junction
-		(at 199.39 73.66)
+		(at 228.6 146.05)
 		(diameter 0)
 		(color 0 0 0 0)
@@
 	)
 	(bus_entry
-		(at 170.18 73.66)
-		(size -2.54 2.54)
+		(at 231.14 73.66)
+		(size 2.54 2.54)
 		(stroke
 			(width 0)
@@
 	)
 	(bus_entry
-		(at 175.26 73.66)
+		(at 170.18 73.66)
 		(size -2.54 2.54)
 		(stroke
@@
 	)
 	(bus_entry
-		(at 246.38 73.66)
-		(size 2.54 2.54)
+		(at 175.26 73.66)
+		(size -2.54 2.54)
 		(stroke
 			(width 0)
@@
 	)
 	(bus_entry
-		(at 233.68 73.66)
+		(at 246.38 73.66)
 		(size 2.54 2.54)
 		(stroke
@@
 	)
 	(bus_entry
-		(at 231.14 73.66)
+		(at 233.68 73.66)
 		(size 2.54 2.54)
 		(stroke
@@
 		)
 	)
-	(wire
+	(bus
 		(pts
-			(xy 99.06 228.6) (xy 99.06 91.44)
+			(xy 199.39 73.66) (xy 228.6 73.66)
 		)
 		(stroke
@@
 	(wire
 		(pts
-			(xy 260.35 184.15) (xy 260.35 187.96)
+			(xy 99.06 228.6) (xy 99.06 91.44)
 		)
 		(stroke
@@
 		)
 	)
-	(bus
+	(wire
 		(pts
-			(xy 199.39 68.58) (xy 199.39 73.66)
+			(xy 260.35 184.15) (xy 260.35 187.96)
 		)
 		(stroke
@@
 	(wire
 		(pts
-			(xy 180.34 91.44) (xy 180.34 86.36)
+			(xy 233.68 76.2) (xy 233.68 91.44)
 		)
 		(stroke
@@
 	(wire
 		(pts
-			(xy 74.93 162.56) (xy 133.35 162.56)
-		)
-		(stroke
-			(width 0)
-			(type default)
-		)
-	)
-	(bus
-		(pts
-			(xy 241.3 73.66) (xy 243.84 73.66)
+			(xy 180.34 91.44) (xy 180.34 86.36)
 		)
 		(stroke
@@
 	(wire
 		(pts
-			(xy 181.61 203.2) (xy 181.61 125.73)
+			(xy 74.93 162.56) (xy 133.35 162.56)
 		)
 		(stroke
@@
 	(bus
 		(pts
-			(xy 231.14 73.66) (xy 233.68 73.66)
+			(xy 241.3 73.66) (xy 243.84 73.66)
 		)
 		(stroke
@@
 	(wire
 		(pts
-			(xy 140.97 44.45) (xy 140.97 46.99)
+			(xy 181.61 203.2) (xy 181.61 125.73)
 		)
 		(stroke
@@
 	(wire
 		(pts
-			(xy 67.31 135.89) (xy 67.31 154.94)
+			(xy 140.97 44.45) (xy 140.97 46.99)
 		)
 		(stroke
@@
 	(wire
 		(pts
-			(xy 233.68 76.2) (xy 233.68 91.44)
+			(xy 67.31 135.89) (xy 67.31 154.94)
 		)
 		(stroke
@@
 		)
 	)
-	(wire
+	(bus
 		(pts
-			(xy 231.14 76.2) (xy 231.14 91.44)
+			(xy 199.39 68.58) (xy 199.39 73.66)
 		)
 		(stroke
@@
 		)
 	)
+	(bus
+		(pts
+			(xy 228.6 73.66) (xy 231.14 73.66)
+		)
+		(stroke
+			(width 0)
+			(type default)
+		)
+	)
 	(wire
 		(pts
@@
 		)
 	)
-	(bus
-		(pts
-			(xy 177.8 73.66) (xy 199.39 73.66)
-		)
-		(stroke
-			(width 0)
-			(type default)
-		)
-	)
 	(wire
 		(pts
@@
 		)
 	)
+	(bus
+		(pts
+			(xy 231.14 73.66) (xy 233.68 73.66)
+		)
+		(stroke
+			(width 0)
+			(type default)
+		)
+	)
 	(wire
 		(pts
@@
 		)
 	)
-	(bus
-		(pts
-			(xy 199.39 73.66) (xy 228.6 73.66)
-		)
-		(stroke
-			(width 0)
-			(type default)
-		)
-	)
 	(wire
 		(pts
@@
 	(bus
 		(pts
-			(xy 228.6 73.66) (xy 231.14 73.66)
-		)
-		(stroke
-			(width 0)
-			(type default)
-		)
-	)
-	(bus
-		(pts
 			(xy 170.18 73.66) (xy 172.72 73.66)
 		)
@@
 	(wire
 		(pts
+			(xy 231.14 76.2) (xy 231.14 91.44)
+		)
+		(stroke
+			(width 0)
+			(type default)
+		)
+	)
+	(wire
+		(pts
 			(xy 88.9 228.6) (xy 99.06 228.6)
 		)
@@
 		)
 	)
+	(bus
+		(pts
+			(xy 177.8 73.66) (xy 199.39 73.66)
+		)
+		(stroke
+			(width 0)
+			(type default)
+		)
+	)
 	(wire
 		(pts
@@
 		)
 	)
-	(label "BTNs4"
-		(at 238.76 77.47 270)
+	(label "BTNs7"
+		(at 231.14 77.47 270)
 		(effects
 			(font
@@
 		)
 	)
-	(label "BTNs0"
-		(at 248.92 77.47 270)
+	(label "BTNs4"
+		(at 238.76 77.47 270)
 		(effects
 			(font
@@
 		)
 	)
-	(label "BTNs8"
-		(at 175.26 77.47 270)
+	(label "BTNs0"
+		(at 248.92 77.47 270)
 		(effects
 			(font
@@
 		)
 	)
-	(label "BTNs2"
-		(at 243.84 77.47 270)
+	(label "BTNs6"
+		(at 233.68 77.47 270)
 		(effects
 			(font
@@
 		)
 	)
-	(label "BTNs3"
-		(at 241.3 77.47 270)
+	(label "BTNs8"
+		(at 175.26 77.47 270)
 		(effects
 			(font
@@
 		)
 	)
-	(label "BTNs5"
-		(at 236.22 77.47 270)
+	(label "BTNs2"
+		(at 243.84 77.47 270)
 		(effects
 			(font
@@
 		)
 	)
-	(label "BTNs10"
-		(at 170.18 77.47 270)
+	(label "BTNs3"
+		(at 241.3 77.47 270)
 		(effects
 			(font
@@
 		)
 	)
-	(label "BTNs6"
-		(at 233.68 77.47 270)
+	(label "BTNs5"
+		(at 236.22 77.47 270)
 		(effects
 			(font
@@
 		)
 	)
-	(label "BTNs7"
-		(at 231.14 77.47 270)
+	(label "BTNs10"
+		(at 170.18 77.47 270)
 		(effects
 			(font
@@
 			)
 		)
-		(pin "BTNs" output
+		(pin "BTNs[0..11]" output
 			(at 199.39 68.58 270)
 			(effects

Commit message: First commit new branch
Connections:
- net BTNs0 renamed BTNs_L0
- net BTNs1 renamed BTNs_L1
- net BTNs10 renamed BTNs_L10
- net BTNs11 renamed BTNs_L11
- net BTNs2 renamed BTNs_L2
- net BTNs3 renamed BTNs_L3
- net BTNs4 renamed BTNs_L4
- net BTNs5 renamed BTNs_L5
- net BTNs6 renamed BTNs_L6
- net BTNs7 renamed BTNs_L7
- net BTNs8 renamed BTNs_L8
- net BTNs9 renamed BTNs_L9
Other:
- removed sheet keyboard
Changed lines of the file:
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@@
 		)
 	)
+	(bus
+		(pts
+			(xy 199.39 34.29) (xy 199.39 73.66)
+		)
+		(stroke
+			(width 0)
+			(type default)
+		)
+	)
 	(wire
 		(pts
@@
 		)
 	)
-	(bus
-		(pts
-			(xy 199.39 68.58) (xy 199.39 73.66)
-		)
-		(stroke
-			(width 0)
-			(type default)
-		)
-	)
 	(wire
 		(pts
@@
 		)
 	)
-	(label "BTNs1"
+	(label "BTNs_L1"
 		(at 246.38 77.47 270)
 		(effects
@@
 		)
 	)
-	(label "BTNs11"
+	(label "BTNs_L11"
 		(at 167.64 77.47 270)
 		(effects
@@
 		)
 	)
-	(label "BTNs9"
+	(label "BTNs_L9"
 		(at 172.72 77.47 270)
 		(effects
@@
 		)
 	)
-	(label "BTNs7"
+	(label "BTNs_L[0..11]"
+		(at 204.47 73.66 0)
+		(effects
+			(font
+				(size 1.27 1.27)
+			)
+			(justify left bottom)
+		)
+	)
+	(label "BTNs_L7"
 		(at 231.14 77.47 270)
 		(effects
@@
 		)
 	)
-	(label "BTNs4"
+	(label "BTNs_L4"
 		(at 238.76 77.47 270)
 		(effects
@@
 		)
 	)
-	(label "BTNs0"
+	(label "BTNs_L0"
 		(at 248.92 77.47 270)
 		(effects
@@
 		)
 	)
-	(label "BTNs6"
+	(label "BTNs_L6"
 		(at 233.68 77.47 270)
 		(effects
@@
 		)
 	)
-	(label "BTNs8"
+	(label "BTNs_L8"
 		(at 175.26 77.47 270)
 		(effects
@@
 		)
 	)
-	(label "BTNs2"
+	(label "BTNs_L2"
 		(at 243.84 77.47 270)
 		(effects
@@
 		)
 	)
-	(label "BTNs3"
+	(label "BTNs_L3"
 		(at 241.3 77.47 270)
 		(effects
@@
 		)
 	)
-	(label "BTNs5"
+	(label "BTNs_L5"
 		(at 236.22 77.47 270)
 		(effects
@@
 		)
 	)
-	(label "BTNs10"
+	(label "BTNs_L10"
 		(at 170.18 77.47 270)
 		(effects
@@
 		)
 	)
+	(hierarchical_label "BTNs_L[0..11]"
+		(shape output)
+		(at 199.39 34.29 90)
+		(effects
+			(font
+				(size 1.27 1.27)
+			)
+			(justify left)
+		)
+	)
 	(hierarchical_label "R_endrow"
 		(shape output)
@@
 		(dnp no)
 		(fields_autoplaced yes)
-		(property "Reference" "#PWR0127"
+		(property "Reference" "#PWR0135"
 			(at 339.09 93.98 0)
 			(effects
@@
 			(project "tastiera_isomorfa"
 				(path "/2a6329ec-b0e8-4012-8f5a-476608b8b2cc/07e251ec-a89a-41e0-b307-1d6ec78f24c5"
-					(reference "#PWR0127")
+					(reference "#PWR0135")
 					(unit 1)
 				)
@@
 		(dnp no)
 		(fields_autoplaced yes)
-		(property "Reference" "#PWR0112"
+		(property "Reference" "#PWR0120"
 			(at 99.06 48.26 0)
 			(effects
@@
 			(project "tastiera_isomorfa"
 				(path "/2a6329ec-b0e8-4012-8f5a-476608b8b2cc/07e251ec-a89a-41e0-b307-1d6ec78f24c5"
-					(reference "#PWR0112")
+					(reference "#PWR0120")
 					(unit 1)
 				)
@@
 		(dnp no)
 		(fields_autoplaced yes)
-		(property "Reference" "#PWR0116"
+		(property "Reference" "#PWR0124"
 			(at 147.32 104.14 0)
 			(effects
@@
 			(project "tastiera_isomorfa"
 				(path "/2a6329ec-b0e8-4012-8f5a-476608b8b2cc/07e251ec-a89a-41e0-b307-1d6ec78f24c5"
-					(reference "#PWR0116")
+					(reference "#PWR0124")
 					(unit 1)
 				)
@@
 		(dnp no)
 		(fields_autoplaced yes)
-		(property "Reference" "#PWR0109"
+		(property "Reference" "#PWR0117"
 			(at 44.45 213.36 0)
 			(effects
@@
 			(project "tastiera_isomorfa"
 				(path "/2a6329ec-b0e8-4012-8f5a-476608b8b2cc/07e251ec-a89a-41e0-b307-1d6ec78f24c5"
-					(reference "#PWR0109")
+					(reference "#PWR0117")
 					(unit 1)
 				)
@@
 		(dnp no)
 		(fields_autoplaced yes)
-		(property "Reference" "#PWR0122"
+		(property "Reference" "#PWR0130"
 			(at 250.19 175.26 0)
 			(effects
@@
 			(project "tastiera_isomorfa"
 				(path "/2a6329ec-b0e8-4012-8f5a-476608b8b2cc/07e251ec-a89a-41e0-b307-1d6ec78f24c5"
-					(reference "#PWR0122")
+					(reference "#PWR0130")
 					(unit 1)
 				)
@@
 		(dnp no)
 		(fields_autoplaced yes)
-		(property "Reference" "#PWR0113"
+		(property "Reference" "#PWR0121"
 			(at 116.84 48.26 0)
 			(effects
@@
 			(project "tastiera_isomorfa"
 				(path "/2a6329ec-b0e8-4012-8f5a-476608b8b2cc/07e251ec-a89a-41e0-b307-1d6ec78f24c5"
-					(reference "#PWR0113")
+					(reference "#PWR0121")
 					(unit 1)
 				)
@@
 		(dnp no)
 		(fields_autoplaced yes)
-		(property "Reference" "#PWR0111"
+		(property "Reference" "#PWR0119"
 			(at 88.9 219.71 0)
 			(effects
@@
 			(project "tastiera_isomorfa"
 				(path "/2a6329ec-b0e8-4012-8f5a-476608b8b2cc/07e251ec-a89a-41e0-b307-1d6ec78f24c5"
-					(reference "#PWR0111")
+					(reference "#PWR0119")
 					(unit 1)
 				)
@@
 		(dnp no)
 		(fields_autoplaced yes)
-		(property "Reference" "#PWR0123"
+		(property "Reference" "#PWR0131"
 			(at 269.24 113.03 0)
 			(effects
@@
 			(project "tastiera_isomorfa"
 				(path "/2a6329ec-b0e8-4012-8f5a-476608b8b2cc/07e251ec-a89a-41e0-b307-1d6ec78f24c5"
-					(reference "#PWR0123")
+					(reference "#PWR0131")
 					(unit 1)
 				)
@@
 		(dnp no)
 		(fields_autoplaced yes)
-		(property "Reference" "#PWR0121"
+		(property "Reference" "#PWR0129"
 			(at 248.92 241.3 0)
 			(effects
@@
 			(project "tastiera_isomorfa"
 				(path "/2a6329ec-b0e8-4012-8f5a-476608b8b2cc/07e251ec-a89a-41e0-b307-1d6ec78f24c5"
-					(reference "#PWR0121")
+					(reference "#PWR0129")
 					(unit 1)
 				)
@@
 		(dnp no)
 		(fields_autoplaced yes)
-		(property "Reference" "#PWR0118"
+		(property "Reference" "#PWR0126"
 			(at 195.58 113.03 0)
 			(effects
@@
 			(project "tastiera_isomorfa"
 				(path "/2a6329ec-b0e8-4012-8f5a-476608b8b2cc/07e251ec-a89a-41e0-b307-1d6ec78f24c5"
-					(reference "#PWR0118")
+					(reference "#PWR0126")
 					(unit 1)
 				)
@@
 		(dnp no)
 		(fields_autoplaced yes)
-		(property "Reference" "#PWR0114"
+		(property "Reference" "#PWR0122"
 			(at 140.97 48.26 0)
 			(effects
@@
 			(project "tastiera_isomorfa"
 				(path "/2a6329ec-b0e8-4012-8f5a-476608b8b2cc/07e251ec-a89a-41e0-b307-1d6ec78f24c5"
-					(reference "#PWR0114")
+					(reference "#PWR0122")
 					(unit 1)
 				)
@@
 		(dnp no)
 		(fields_autoplaced yes)
-		(property "Reference" "#PWR0124"
+		(property "Reference" "#PWR0132"
 			(at 270.51 182.88 0)
 			(effects
@@
 			(project "tastiera_isomorfa"
 				(path "/2a6329ec-b0e8-4012-8f5a-476608b8b2cc/07e251ec-a89a-41e0-b307-1d6ec78f24c5"
-					(reference "#PWR0124")
+					(reference "#PWR0132")
 					(unit 1)
 				)
@@
 		(dnp no)
 		(fields_autoplaced yes)
-		(property "Reference" "#PWR0119"
+		(property "Reference" "#PWR0127"
 			(at 220.98 104.14 0)
 			(effects
@@
 			(project "tastiera_isomorfa"
 				(path "/2a6329ec-b0e8-4012-8f5a-476608b8b2cc/07e251ec-a89a-41e0-b307-1d6ec78f24c5"
-					(reference "#PWR0119")
+					(reference "#PWR0127")
 					(unit 1)
 				)
@@
 		(dnp no)
 		(fields_autoplaced yes)
-		(property "Reference" "#PWR0125"
+		(property "Reference" "#PWR0133"
 			(at 326.39 59.69 0)
 			(effects
@@
 			(project "tastiera_isomorfa"
 				(path "/2a6329ec-b0e8-4012-8f5a-476608b8b2cc/07e251ec-a89a-41e0-b307-1d6ec78f24c5"
-					(reference "#PWR0125")
+					(reference "#PWR0133")
 					(unit 1)
 				)
@@
 		(dnp no)
 		(fields_autoplaced yes)
-		(property "Reference" "#PWR0110"
+		(property "Reference" "#PWR0118"
 			(at 63.5 64.77 0)
 			(effects
@@
 			(project "tastiera_isomorfa"
 				(path "/2a6329ec-b0e8-4012-8f5a-476608b8b2cc/07e251ec-a89a-41e0-b307-1d6ec78f24c5"
-					(reference "#PWR0110")
+					(reference "#PWR0118")
 					(unit 1)
 				)
@@
 		(dnp no)
 		(fields_autoplaced yes)
-		(property "Reference" "#PWR0117"
+		(property "Reference" "#PWR0125"
 			(at 162.56 77.47 0)
 			(effects
@@
 			(project "tastiera_isomorfa"
 				(path "/2a6329ec-b0e8-4012-8f5a-476608b8b2cc/07e251ec-a89a-41e0-b307-1d6ec78f24c5"
-					(reference "#PWR0117")
+					(reference "#PWR0125")
 					(unit 1)
 				)
@@
 		(dnp no)
 		(fields_autoplaced yes)
-		(property "Reference" "#PWR0126"
+		(property "Reference" "#PWR0134"
 			(at 327.66 140.97 0)
 			(effects
@@
 			(project "tastiera_isomorfa"
 				(path "/2a6329ec-b0e8-4012-8f5a-476608b8b2cc/07e251ec-a89a-41e0-b307-1d6ec78f24c5"
-					(reference "#PWR0126")
+					(reference "#PWR0134")
 					(unit 1)
 				)
@@
 		(dnp no)
 		(fields_autoplaced yes)
-		(property "Reference" "#PWR0120"
+		(property "Reference" "#PWR0128"
 			(at 237.49 241.3 0)
 			(effects
@@
 			(project "tastiera_isomorfa"
 				(path "/2a6329ec-b0e8-4012-8f5a-476608b8b2cc/07e251ec-a89a-41e0-b307-1d6ec78f24c5"
-					(reference "#PWR0120")
+					(reference "#PWR0128")
 					(unit 1)
 				)
@@
 		(dnp no)
 		(fields_autoplaced yes)
-		(property "Reference" "#PWR0115"
+		(property "Reference" "#PWR0123"
 			(at 144.78 242.57 0)
 			(effects
@@
 			(project "tastiera_isomorfa"
 				(path "/2a6329ec-b0e8-4012-8f5a-476608b8b2cc/07e251ec-a89a-41e0-b307-1d6ec78f24c5"
-					(reference "#PWR0115")
+					(reference "#PWR0123")
 					(unit 1)
 				)
@@
 				)
 			)
-		)
-	)
-	(sheet
-		(at 170.18 55.88)
-		(size 58.42 12.7)
-		(exclude_from_sim no)
-		(in_bom yes)
-		(on_board yes)
-		(dnp no)
-		(fields_autoplaced yes)
-		(stroke
-			(width 0.1524)
-			(type solid)
-		)
-		(fill
-			(color 0 0 0 0.0000)
-		)
-		(property "Sheetname" "keyboard"
-			(at 170.18 55.1684 0)
-			(effects
-				(font
-					(size 1.27 1.27)
-				)
-				(justify left bottom)
-			)
-		)
-		(property "Sheetfile" "keyboard.kicad_sch"
-			(at 170.18 69.1646 0)
-			(effects
-				(font
-					(size 1.27 1.27)
-				)
-				(justify left top)
-			)
-		)
-		(pin "BTNs[0..11]" output
-			(at 199.39 68.58 270)
-			(effects
-				(font
-					(size 1.27 1.27)
-				)
-				(justify left)
-			)
-		)
-		(instances
-			(project "tastiera_isomorfa"
-				(path "/2a6329ec-b0e8-4012-8f5a-476608b8b2cc/07e251ec-a89a-41e0-b307-1d6ec78f24c5"
-					(page "4")
-				)
-			)
