File: hardware/kicad/module-tile/tastiera_isomorfa.kicad_sch (KiCad schematic)
At the start: 8 parts, among them J101 Conn_LEFT, J102 Conn_TOP, J103 Conn_BOTTOM, J104 Conn_RIGHT, J105 BTNs_L_MSB, J106 BTNs_L_LSB, J107 BTNs_MSB, J108 BTNs_LSB

Commit message: Adjust interboard pitch
Parts:
- J101, J102: Codice (none) -> 613010143121; Link (none) -> https://www.digikey.it/it/products/detail/w%C3%BCrth-elektr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
- J103, J104: Codice (none) -> 61300811021; Link (none) -> https://www.digikey.it/it/products/detail/w%C3%BCrth-elektr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
Changed lines of the file:
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@@
 			)
 		)
-		(property "Codice" ""
+		(property "Codice" "613010143121"
 			(at 87.63 69.85 90)
 			(effects
@@
 			)
 		)
-		(property "Link" ""
+		(property "Link" "https://www.digikey.it/it/products/detail/w%C3%BCrth-elektronik/613010143121/2508632"
 			(at 87.63 69.85 90)
 			(effects
@@
 			)
 		)
-		(property "Codice" ""
+		(property "Codice" "613010143121"
 			(at 36.83 120.65 0)
 			(effects
@@
 			)
 		)
-		(property "Link" ""
+		(property "Link" "https://www.digikey.it/it/products/detail/w%C3%BCrth-elektronik/613010143121/2508632"
 			(at 36.83 120.65 0)
 			(effects
@@
 			)
 		)
-		(property "Codice" ""
+		(property "Codice" "61300811021"
 			(at 140.97 120.65 0)
 			(effects
@@
 			)
 		)
-		(property "Link" ""
+		(property "Link" "https://www.digikey.it/it/products/detail/w%C3%BCrth-elektronik/61300811021/4846838"
 			(at 140.97 120.65 0)
 			(effects
@@
 			)
 		)
-		(property "Codice" ""
+		(property "Codice" "61300811021"
 			(at 87.63 173.99 90)
 			(effects
@@
 			)
 		)
-		(property "Link" ""
+		(property "Link" "https://www.digikey.it/it/products/detail/w%C3%BCrth-elektronik/61300811021/4846838"
 			(at 87.63 173.99 90)
 			(effects
