File: hardware/kicad/tile/counter.kicad_sch (KiCad schematic)
At the start: 4 parts, among them U102 74AUC2G08, U106 74LVC2G32, U108 74LVC2G74, U109 74LS161

Commit message: KiCad: rename Italian field and footprint names
- Symbol field "Codice" (manufacturer part number) -> "MPN".
- Mouse-bite footprint "Senza-titolo" -> "MouseBite_NPTH_0.5mm".

Verified: netlist identical to rev A, switch/connector/outline
invariants OK, DRC report counts unchanged.
Parts:
- U102: Codice SN74LVC2G08IDCTRQ1 -> (none); MPN (none) -> SN74LVC2G08IDCTRQ1
- U106: Codice SN74LVC2G32DCTR -> (none); MPN (none) -> SN74LVC2G32DCTR
- U108: Codice SN74LVC2G74DCTR -> (none); MPN (none) -> SN74LVC2G74DCTR
- U109: Codice SN74HC161DR -> (none); MPN (none) -> SN74HC161DR
Changed lines of the file:
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@@
 			)
 		)
-		(property "Codice" "SN74LVC2G32DCTR"
+		(property "MPN" "SN74LVC2G32DCTR"
 			(at 110.49 96.52 0)
 			(effects
@@
 			)
 		)
-		(property "Codice" "SN74LVC2G74DCTR"
+		(property "MPN" "SN74LVC2G74DCTR"
 			(at 66.04 93.98 0)
 			(effects
@@
 			)
 		)
-		(property "Codice" "SN74LVC2G08IDCTRQ1"
+		(property "MPN" "SN74LVC2G08IDCTRQ1"
 			(at 156.21 93.98 0)
 			(effects
@@
 			)
 		)
-		(property "Codice" "SN74HC161DR"
+		(property "MPN" "SN74HC161DR"
 			(at 195.58 109.22 0)
 			(effects

Commit message: Rev B schematic: series termination, decoupling, assembly-ready parts
Function unchanged (no logic connection changes). Applied by
hardware/kicad/tile/scripts/revb_schematic.py:

- 33 ohm series resistors R201-R207 at every driver leaving the tile
  (L_clk, T_clk, L_latch, T_latch, B_data, R_data, B_W).
- 100 nF per logic IC (C201-C209); PWR_FLAGs on VCC, GND, VCC_T, GND_T.
- Values match the ordered parts (74LVC..., 74HC161); footprints:
  0603 passives, TI DCT land pattern for the 2G parts, standard
  SOT-23-5, SMD bulk capacitor, Kailh MX hot-swap sockets; Manufacturer
  and MPN fields, Link field dropped.
- Project footprint library with the hot-swap socket from
  keyswitch-kicad-library v2.3 (CC-BY-SA 4.0 with design exception).

Verified: netlist identical to rev A after collapsing R201-R207 and
ignoring C201-C209; ERC 0 errors (was 4).
Parts:
- U102: value 74AUC2G08 -> 74LVC2G08; footprint Package_SO:MSOP-8_3x3mm_P0.65mm -> Package_SO:SSOP-8_2.95x2.8mm_P0.65mm; Link https://www.digikey.it/it/products/detail/texas-instruments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 -> (none); MPN SN74LVC2G08IDCTRQ1 -> SN74LVC2G08DCTR; Manufacturer (none) -> Texas Instruments
- U106, U108: footprint Package_SO:MSOP-8_3x3mm_P0.65mm -> Package_SO:SSOP-8_2.95x2.8mm_P0.65mm; Link https://www.digikey.it/it/products/detail/texas-instruments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 -> (none); Manufacturer (none) -> Texas Instruments
- U109: value 74LS161 -> 74HC161; Link https://www.digikey.it/it/products/detail/texas-instruments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 -> (none); Manufacturer (none) -> Texas Instruments
Changed lines of the file:
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@@
 			)
 		)
-		(property "Footprint" "Package_SO:MSOP-8_3x3mm_P0.65mm"
+		(property "Footprint" "Package_SO:SSOP-8_2.95x2.8mm_P0.65mm"
 			(at 110.49 96.52 0)
 			(hide yes)
@@
 			)
 		)
+		(property "Manufacturer" "Texas Instruments"
+			(at 110.49 96.52 0)
+			(hide yes)
+			(show_name no)
+			(do_not_autoplace no)
+			(effects
+				(font
+					(size 1.27 1.27)
+				)
+			)
+		)
 		(property "MPN" "SN74LVC2G32DCTR"
-			(at 110.49 96.52 0)
-			(hide yes)
-			(show_name no)
-			(do_not_autoplace no)
-			(effects
-				(font
-					(size 1.27 1.27)
-				)
-			)
-		)
-		(property "Link" "https://www.digikey.it/it/products/detail/texas-instruments/SN74LVC2G32DCTR/484828"
 			(at 110.49 96.52 0)
 			(hide yes)
@@
 			)
 		)
-		(property "Footprint" "Package_SO:MSOP-8_3x3mm_P0.65mm"
+		(property "Footprint" "Package_SO:SSOP-8_2.95x2.8mm_P0.65mm"
 			(at 66.04 93.98 0)
 			(hide yes)
@@
 			)
 		)
+		(property "Manufacturer" "Texas Instruments"
+			(at 66.04 93.98 0)
+			(hide yes)
+			(show_name no)
+			(do_not_autoplace no)
+			(effects
+				(font
+					(size 1.27 1.27)
+				)
+			)
+		)
 		(property "MPN" "SN74LVC2G74DCTR"
-			(at 66.04 93.98 0)
-			(hide yes)
-			(show_name no)
-			(do_not_autoplace no)
-			(effects
-				(font
-					(size 1.27 1.27)
-				)
-			)
-		)
-		(property "Link" "https://www.digikey.it/it/products/detail/texas-instruments/SN74LVC2G74DCTR/484721"
 			(at 66.04 93.98 0)
 			(hide yes)
@@
 			)
 		)
-		(property "Value" "74AUC2G08"
+		(property "Value" "74LVC2G08"
 			(at 157.4911 86.36 0)
 			(show_name no)
@@
 			)
 		)
-		(property "Footprint" "Package_SO:MSOP-8_3x3mm_P0.65mm"
+		(property "Footprint" "Package_SO:SSOP-8_2.95x2.8mm_P0.65mm"
 			(at 156.21 93.98 0)
 			(hide yes)
@@
 			)
 		)
-		(property "MPN" "SN74LVC2G08IDCTRQ1"
+		(property "Manufacturer" "Texas Instruments"
 			(at 156.21 93.98 0)
 			(hide yes)
@@
 			)
 		)
-		(property "Link" "https://www.digikey.it/it/products/detail/texas-instruments/SN74LVC2G08IDCTRQ1/1592267"
+		(property "MPN" "SN74LVC2G08DCTR"
 			(at 156.21 93.98 0)
 			(hide yes)
@@
 			)
 		)
-		(property "Value" "74LS161"
+		(property "Value" "74HC161"
 			(at 193.4367 78.74 0)
 			(show_name no)
@@
 			)
 		)
+		(property "Manufacturer" "Texas Instruments"
+			(at 195.58 109.22 0)
+			(hide yes)
+			(show_name no)
+			(do_not_autoplace no)
+			(effects
+				(font
+					(size 1.27 1.27)
+				)
+			)
+		)
 		(property "MPN" "SN74HC161DR"
 			(at 195.58 109.22 0)
 			(hide yes)
-			(show_name no)
-			(do_not_autoplace no)
-			(effects
-				(font
-					(size 1.27 1.27)
-				)
-			)
-		)
-		(property "Link" "https://www.digikey.it/it/products/detail/texas-instruments/SN74HC161DR/562878"
-			(at 195.58 109.22 0)
-			(hide yes)
