File: hardware/kicad/tile/power.kicad_sch (KiCad schematic)
At the start: 9 parts, among them U101 74AUC2G126, U102 74AUC2G08, U106 74LVC2G32, U107 74AUC2G125

Commit message: KiCad: rename Italian field and footprint names
- Symbol field "Codice" (manufacturer part number) -> "MPN".
- Mouse-bite footprint "Senza-titolo" -> "MouseBite_NPTH_0.5mm".

Verified: netlist identical to rev A, switch/connector/outline
invariants OK, DRC report counts unchanged.
Parts:
- C101, C102: Codice C0805C104K5RACTU -> (none); MPN (none) -> C0805C104K5RACTU
- C103, C104: Codice CL31B475KAHNNNE -> (none); MPN (none) -> CL31B475KAHNNNE
- C105: Codice 860040573004 -> (none); MPN (none) -> 860040573004
- U101: Codice 74LVC2G126DCTRG4 -> (none); MPN (none) -> 74LVC2G126DCTRG4
- U102: Codice SN74LVC2G08IDCTRQ1 -> (none); MPN (none) -> SN74LVC2G08IDCTRQ1
- U106: Codice SN74LVC2G32DCTR -> (none); MPN (none) -> SN74LVC2G32DCTR
- U107: Codice SN74LVC2G125DCTR -> (none); MPN (none) -> SN74LVC2G125DCTR
Changed lines of the file:
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@@
 			)
 		)
-		(property "Codice" "74LVC2G126DCTRG4"
+		(property "MPN" "74LVC2G126DCTRG4"
 			(at 187.96 72.39 0)
 			(effects
@@
 			)
 		)
-		(property "Codice" "CL31B475KAHNNNE"
+		(property "MPN" "CL31B475KAHNNNE"
 			(at 170.18 127 0)
 			(effects
@@
 			)
 		)
-		(property "Codice" "SN74LVC2G08IDCTRQ1"
+		(property "MPN" "SN74LVC2G08IDCTRQ1"
 			(at 99.06 72.39 0)
 			(effects
@@
 			)
 		)
-		(property "Codice" "SN74LVC2G125DCTR"
+		(property "MPN" "SN74LVC2G125DCTR"
 			(at 160.02 72.39 0)
 			(effects
@@
 			)
 		)
-		(property "Codice" "C0805C104K5RACTU"
+		(property "MPN" "C0805C104K5RACTU"
 			(at 119.38 127 0)
 			(effects
@@
 			)
 		)
-		(property "Codice" "CL31B475KAHNNNE"
+		(property "MPN" "CL31B475KAHNNNE"
 			(at 144.78 127 0)
 			(effects
@@
 			)
 		)
-		(property "Codice" "C0805C104K5RACTU"
+		(property "MPN" "C0805C104K5RACTU"
 			(at 93.98 127 0)
 			(effects
@@
 			)
 		)
-		(property "Codice" "860040573004"
+		(property "MPN" "860040573004"
 			(at 195.58 127 0)
 			(effects
@@
 			)
 		)
-		(property "Codice" "SN74LVC2G32DCTR"
+		(property "MPN" "SN74LVC2G32DCTR"
 			(at 130.81 72.39 0)
 			(effects

Commit message: Rev B schematic: series termination, decoupling, assembly-ready parts
Function unchanged (no logic connection changes). Applied by
hardware/kicad/tile/scripts/revb_schematic.py:

- 33 ohm series resistors R201-R207 at every driver leaving the tile
  (L_clk, T_clk, L_latch, T_latch, B_data, R_data, B_W).
- 100 nF per logic IC (C201-C209); PWR_FLAGs on VCC, GND, VCC_T, GND_T.
- Values match the ordered parts (74LVC..., 74HC161); footprints:
  0603 passives, TI DCT land pattern for the 2G parts, standard
  SOT-23-5, SMD bulk capacitor, Kailh MX hot-swap sockets; Manufacturer
  and MPN fields, Link field dropped.
- Project footprint library with the hot-swap socket from
  keyswitch-kicad-library v2.3 (CC-BY-SA 4.0 with design exception).

Verified: netlist identical to rev A after collapsing R201-R207 and
ignoring C201-C209; ERC 0 errors (was 4).
Parts:
- added C201, C202, C203, C204, C205, C206, C207, C208, C209: 100n, Capacitor_SMD:C_0603_1608Metric, symbol Device:C
- C101, C102: footprint Capacitor_SMD:C_0805_2012Metric_Pad1.18x1.45mm_HandSolder -> Capacitor_SMD:C_0603_1608Metric; Link https://www.digikey.it/it/products/detail/kemet/C0805C104K5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 -> (none); MPN C0805C104K5RACTU -> CL10B104KB8NNNC; Manufacturer (none) -> Samsung
- C103, C104: footprint Capacitor_SMD:C_1206_3216Metric_Pad1.33x1.80mm_HandSolder -> Capacitor_SMD:C_1206_3216Metric; Link https://www.digikey.it/it/products/detail/samsung-electro-m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 -> (none); Manufacturer (none) -> Samsung
- C105: footprint Capacitor_THT:CP_Radial_D6.3mm_P2.50mm -> Capacitor_SMD:CP_Elec_6.3x7.7; Link https://www.digikey.it/it/products/detail/w%C3%BCrth-elektr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 -> (none); MPN 860040573004 -> (none)
- U101: value 74AUC2G126 -> 74LVC2G126; footprint Package_SO:MSOP-8_3x3mm_P0.65mm -> Package_SO:SSOP-8_2.95x2.8mm_P0.65mm; Link https://www.digikey.it/it/products/detail/texas-instruments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 -> (none); MPN 74LVC2G126DCTRG4 -> SN74LVC2G126DCTR; Manufacturer (none) -> Texas Instruments
- U102: value 74AUC2G08 -> 74LVC2G08; footprint Package_SO:MSOP-8_3x3mm_P0.65mm -> Package_SO:SSOP-8_2.95x2.8mm_P0.65mm; Link https://www.digikey.it/it/products/detail/texas-instruments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 -> (none); MPN SN74LVC2G08IDCTRQ1 -> SN74LVC2G08DCTR; Manufacturer (none) -> Texas Instruments
- U106: footprint Package_SO:MSOP-8_3x3mm_P0.65mm -> Package_SO:SSOP-8_2.95x2.8mm_P0.65mm; Link https://www.digikey.it/it/products/detail/texas-instruments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 -> (none); Manufacturer (none) -> Texas Instruments
- U107: value 74AUC2G125 -> 74LVC2G125; footprint Package_SO:MSOP-8_3x3mm_P0.65mm -> Package_SO:SSOP-8_2.95x2.8mm_P0.65mm; Link https://www.digikey.it/it/products/detail/texas-instruments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 -> (none); Manufacturer (none) -> Texas Instruments
Connections:
- net GND: now also C201.2, C202.2, C203.2, C204.2, C205.2, C206.2, C207.2, C208.2, C209.2
- net VCC: now also C201.1, C202.1, C203.1, C204.1, C205.1, C206.1, C207.1, C208.1, C209.1
Other:
- note added: "Rev B: one 100 nF (0603) per logic IC, placed next to its VCC pin on the PCB: C201 U101, C202 U102, C203 U103, C204 U104, C205 U105, C206 U106, C207 U107, C208 U108, C209 U109"
