File: hardware/kicad/tile/tile.kicad_sch (KiCad schematic)
At the start: 16 parts, among them U101 74AUC2G126, U102 74AUC2G08, U103 74HC165, U104 74HC165, U105 74AHC1G04, U106 74LVC2G32, U107 74AUC2G125

Commit message: KiCad: rename Italian field and footprint names
- Symbol field "Codice" (manufacturer part number) -> "MPN".
- Mouse-bite footprint "Senza-titolo" -> "MouseBite_NPTH_0.5mm".

Verified: netlist identical to rev A, switch/connector/outline
invariants OK, DRC report counts unchanged.
Parts:
- R101, R102, R103, R104, R105, R106, R107, R108, R109: Codice RMCF0805FT10K0 -> (none); MPN (none) -> RMCF0805FT10K0
- U101: Codice 74LVC2G126DCTRG4 -> (none); MPN (none) -> 74LVC2G126DCTRG4
- U102: Codice SN74LVC2G08IDCTRQ1 -> (none); MPN (none) -> SN74LVC2G08IDCTRQ1
- U103, U104: Codice SN74LVC165ADR -> (none); MPN (none) -> SN74LVC165ADR
- U105: Codice SN74LVC1G04DBVR -> (none); MPN (none) -> SN74LVC1G04DBVR
- U106: Codice SN74LVC2G32DCTR -> (none); MPN (none) -> SN74LVC2G32DCTR
- U107: Codice SN74LVC2G125DCTR -> (none); MPN (none) -> SN74LVC2G125DCTR
Changed lines of the file:
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@@
 			)
 		)
-		(property "Codice" "SN74LVC2G32DCTR"
+		(property "MPN" "SN74LVC2G32DCTR"
 			(at 260.35 200.66 90)
 			(effects
@@
 			)
 		)
-		(property "Codice" "SN74LVC165ADR"
+		(property "MPN" "SN74LVC165ADR"
 			(at 243.84 104.14 90)
 			(effects
@@
 			)
 		)
-		(property "Codice" "RMCF0805FT10K0"
+		(property "MPN" "RMCF0805FT10K0"
 			(at 140.97 50.8 0)
 			(effects
@@
 			)
 		)
-		(property "Codice" "SN74LVC1G04DBVR"
+		(property "MPN" "SN74LVC1G04DBVR"
 			(at 260.35 168.91 90)
 			(effects
@@
 			)
 		)
-		(property "Codice" "RMCF0805FT10K0"
+		(property "MPN" "RMCF0805FT10K0"
 			(at 237.49 228.6 0)
 			(effects
@@
 			)
 		)
-		(property "Codice" "RMCF0805FT10K0"
+		(property "MPN" "RMCF0805FT10K0"
 			(at 327.66 143.51 0)
 			(effects
@@
 			)
 		)
-		(property "Codice" "SN74LVC2G08IDCTRQ1"
+		(property "MPN" "SN74LVC2G08IDCTRQ1"
 			(at 109.22 109.22 0)
 			(effects
@@
 			)
 		)
-		(property "Codice" "RMCF0805FT10K0"
+		(property "MPN" "RMCF0805FT10K0"
 			(at 248.92 228.6 0)
 			(effects
@@
 			)
 		)
-		(property "Codice" "RMCF0805FT10K0"
+		(property "MPN" "RMCF0805FT10K0"
 			(at 44.45 200.66 0)
 			(effects
@@
 			)
 		)
-		(property "Codice" "RMCF0805FT10K0"
+		(property "MPN" "RMCF0805FT10K0"
 			(at 326.39 46.99 0)
 			(effects
@@
 			)
 		)
-		(property "Codice" "RMCF0805FT10K0"
+		(property "MPN" "RMCF0805FT10K0"
 			(at 116.84 50.8 0)
 			(effects
@@
 			)
 		)
-		(property "Codice" "RMCF0805FT10K0"
+		(property "MPN" "RMCF0805FT10K0"
 			(at 63.5 67.31 0)
 			(effects
@@
 			)
 		)
-		(property "Codice" "SN74LVC165ADR"
+		(property "MPN" "SN74LVC165ADR"
 			(at 170.18 104.14 90)
 			(effects
@@
 			)
 		)
-		(property "Codice" "RMCF0805FT10K0"
+		(property "MPN" "RMCF0805FT10K0"
 			(at 88.9 222.25 0)
 			(effects
@@
 			)
 		)
-		(property "Codice" "SN74LVC2G125DCTR"
+		(property "MPN" "SN74LVC2G125DCTR"
 			(at 295.91 72.39 0)
 			(effects
@@
 			)
 		)
-		(property "Codice" "74LVC2G126DCTRG4"
+		(property "MPN" "74LVC2G126DCTRG4"
 			(at 62.23 162.56 0)
 			(effects
@@
 			)
 		)
-		(property "Codice" "74LVC2G126DCTRG4"
+		(property "MPN" "74LVC2G126DCTRG4"
 			(at 81.28 151.13 0)
 			(effects
@@
 			)
 		)
-		(property "Codice" "SN74LVC2G125DCTR"
+		(property "MPN" "SN74LVC2G125DCTR"
 			(at 309.88 53.34 0)
 			(effects

Commit message: Rev B schematic: series termination, decoupling, assembly-ready parts
Function unchanged (no logic connection changes). Applied by
hardware/kicad/tile/scripts/revb_schematic.py:

- 33 ohm series resistors R201-R207 at every driver leaving the tile
  (L_clk, T_clk, L_latch, T_latch, B_data, R_data, B_W).
- 100 nF per logic IC (C201-C209); PWR_FLAGs on VCC, GND, VCC_T, GND_T.
- Values match the ordered parts (74LVC..., 74HC161); footprints:
  0603 passives, TI DCT land pattern for the 2G parts, standard
  SOT-23-5, SMD bulk capacitor, Kailh MX hot-swap sockets; Manufacturer
  and MPN fields, Link field dropped.
- Project footprint library with the hot-swap socket from
  keyswitch-kicad-library v2.3 (CC-BY-SA 4.0 with design exception).

Verified: netlist identical to rev A after collapsing R201-R207 and
ignoring C201-C209; ERC 0 errors (was 4).
Parts:
- added R201, R202, R203, R204, R205, R206, R207: 33, Resistor_SMD:R_0603_1608Metric, symbol Device:R
- R101, R102, R103, R104, R105, R106, R107, R108, R109: footprint Resistor_SMD:R_0805_2012Metric_Pad1.20x1.40mm_HandSolder -> Resistor_SMD:R_0603_1608Metric; Link https://www.digikey.it/it/products/detail/stackpole-electro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 -> (none); MPN RMCF0805FT10K0 -> RC0603FR-0710KL; Manufacturer (none) -> Yageo
- U101: value 74AUC2G126 -> 74LVC2G126; footprint Package_SO:MSOP-8_3x3mm_P0.65mm -> Package_SO:SSOP-8_2.95x2.8mm_P0.65mm; Link https://www.digikey.it/it/products/detail/texas-instruments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 -> (none); MPN 74LVC2G126DCTRG4 -> SN74LVC2G126DCTR; Manufacturer (none) -> Texas Instruments
- U102: value 74AUC2G08 -> 74LVC2G08; footprint Package_SO:MSOP-8_3x3mm_P0.65mm -> Package_SO:SSOP-8_2.95x2.8mm_P0.65mm; Link https://www.digikey.it/it/products/detail/texas-instruments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 -> (none); MPN SN74LVC2G08IDCTRQ1 -> SN74LVC2G08DCTR; Manufacturer (none) -> Texas Instruments
- U103, U104: value 74HC165 -> 74LVC165A; Link https://www.digikey.it/it/products/detail/texas-instruments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 -> (none); Manufacturer (none) -> Texas Instruments
- U105: value 74AHC1G04 -> 74LVC1G04; footprint Package_TO_SOT_SMD:SOT-23-5_HandSoldering -> Package_TO_SOT_SMD:SOT-23-5; Link https://www.digikey.it/it/products/detail/texas-instruments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 -> (none); Manufacturer (none) -> Texas Instruments
- U106: footprint Package_SO:MSOP-8_3x3mm_P0.65mm -> Package_SO:SSOP-8_2.95x2.8mm_P0.65mm; Link https://www.digikey.it/it/products/detail/texas-instruments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 -> (none); Manufacturer (none) -> Texas Instruments
- U107: value 74AUC2G125 -> 74LVC2G125; footprint Package_SO:MSOP-8_3x3mm_P0.65mm -> Package_SO:SSOP-8_2.95x2.8mm_P0.65mm; Link https://www.digikey.it/it/products/detail/texas-instruments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 -> (none); Manufacturer (none) -> Texas Instruments
Connections:
- net B_W: now also R207.2
- net B_data: now also R205.2; no longer U104.9 (Q7)
- net L_clk: now also R201.2; no longer U101.6
- net L_latch: now also R203.2; no longer U105.2, U106.7
- net T_clk: now also R202.2; no longer U107.6
- new net B_W_drv: R207.1
- new net L_clk_drv: R201.1, U101.6
- new net R_data: R206.2
- new net T_clk_drv: R202.1, U107.6
- new net T_latch: R204.2
- new net data_drv: R205.1, R206.1, U104.9 (Q7)
- new net latch_drv: R203.1, R204.1, U105.2, U106.7
Other:
- note added: "Rev B: series source termination (33 ohm) on every driver leaving the tile. SI analysis: hardware/si/, docs/architecture/electrical.md"
