File: hardware/kicad/tile/keyboard.kicad_sch (KiCad schematic)
At the start: 36 parts, among them SW101 SW_Push, SW102 SW_Push, SW103 SW_Push, SW104 SW_Push, SW105 SW_Push, SW106 SW_Push, SW107 SW_Push, SW108 SW_Push, SW109 SW_Push, SW110 SW_Push, SW111 SW_Push, SW112 SW_Push

Commit message: KiCad: rename Italian field and footprint names
- Symbol field "Codice" (manufacturer part number) -> "MPN".
- Mouse-bite footprint "Senza-titolo" -> "MouseBite_NPTH_0.5mm".

Verified: netlist identical to rev A, switch/connector/outline
invariants OK, DRC report counts unchanged.
Parts:
- R110, R111, R112, R113, R114, R115, R116, R117, R118, R119, R120, R121: Codice CRCW0805100RFKEA -> (none); MPN (none) -> CRCW0805100RFKEA
- R122, R123, R124, R125, R126, R127, R128, R129, R130, R131, R132, R133: Codice RMCF0805FT10K0 -> (none); MPN (none) -> RMCF0805FT10K0
Changed lines of the file:
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@@
 			)
 		)
-		(property "Codice" "CRCW0805100RFKEA"
+		(property "MPN" "CRCW0805100RFKEA"
 			(at 142.24 41.91 90)
 			(effects
@@
 			)
 		)
-		(property "Codice" "CRCW0805100RFKEA"
+		(property "MPN" "CRCW0805100RFKEA"
 			(at 142.24 153.67 90)
 			(effects
@@
 			)
 		)
-		(property "Codice" ""
+		(property "MPN" ""
 			(at 125.73 72.39 0)
 			(effects
@@
 			)
 		)
-		(property "Codice" ""
+		(property "MPN" ""
 			(at 125.73 62.23 0)
 			(effects
@@
 			)
 		)
-		(property "Codice" "CRCW0805100RFKEA"
+		(property "MPN" "CRCW0805100RFKEA"
 			(at 142.24 72.39 90)
 			(effects
@@
 			)
 		)
-		(property "Codice" "CRCW0805100RFKEA"
+		(property "MPN" "CRCW0805100RFKEA"
 			(at 142.24 123.19 90)
 			(effects
@@
 			)
 		)
-		(property "Codice" "CRCW0805100RFKEA"
+		(property "MPN" "CRCW0805100RFKEA"
 			(at 142.24 143.51 90)
 			(effects
@@
 			)
 		)
-		(property "Codice" "RMCF0805FT10K0"
+		(property "MPN" "RMCF0805FT10K0"
 			(at 172.72 137.16 90)
 			(effects
@@
 			)
 		)
-		(property "Codice" ""
+		(property "MPN" ""
 			(at 125.73 113.03 0)
 			(effects
@@
 			)
 		)
-		(property "Codice" "RMCF0805FT10K0"
+		(property "MPN" "RMCF0805FT10K0"
 			(at 172.72 96.52 90)
 			(effects
@@
 			)
 		)
-		(property "Codice" "CRCW0805100RFKEA"
+		(property "MPN" "CRCW0805100RFKEA"
 			(at 142.24 62.23 90)
 			(effects
@@
 			)
 		)
-		(property "Codice" "CRCW0805100RFKEA"
+		(property "MPN" "CRCW0805100RFKEA"
 			(at 142.24 113.03 90)
 			(effects
@@
 			)
 		)
-		(property "Codice" "CRCW0805100RFKEA"
+		(property "MPN" "CRCW0805100RFKEA"
 			(at 142.24 82.55 90)
 			(effects
@@
 			)
 		)
-		(property "Codice" ""
+		(property "MPN" ""
 			(at 125.73 133.35 0)
 			(effects
@@
 			)
 		)
-		(property "Codice" ""
+		(property "MPN" ""
 			(at 125.73 52.07 0)
 			(effects
@@
 			)
 		)
-		(property "Codice" ""
+		(property "MPN" ""
 			(at 125.73 102.87 0)
 			(effects
@@
 			)
 		)
-		(property "Codice" "RMCF0805FT10K0"
+		(property "MPN" "RMCF0805FT10K0"
 			(at 172.72 106.68 90)
 			(effects
@@
 			)
 		)
-		(property "Codice" "RMCF0805FT10K0"
+		(property "MPN" "RMCF0805FT10K0"
 			(at 172.72 66.04 90)
 			(effects
@@
 			)
 		)
-		(property "Codice" "CRCW0805100RFKEA"
+		(property "MPN" "CRCW0805100RFKEA"
 			(at 142.24 92.71 90)
 			(effects
@@
 			)
 		)
-		(property "Codice" ""
+		(property "MPN" ""
 			(at 125.73 153.67 0)
 			(effects
@@
 			)
 		)
-		(property "Codice" ""
+		(property "MPN" ""
 			(at 125.73 41.91 0)
 			(effects
@@
 			)
 		)
-		(property "Codice" ""
+		(property "MPN" ""
 			(at 125.73 92.71 0)
 			(effects
@@
 			)
 		)
-		(property "Codice" "RMCF0805FT10K0"
+		(property "MPN" "RMCF0805FT10K0"
 			(at 172.72 127 90)
 			(effects
@@
 			)
 		)
-		(property "Codice" "RMCF0805FT10K0"
+		(property "MPN" "RMCF0805FT10K0"
 			(at 172.72 55.88 90)
 			(effects
@@
 			)
 		)
-		(property "Codice" "RMCF0805FT10K0"
+		(property "MPN" "RMCF0805FT10K0"
 			(at 172.72 76.2 90)
 			(effects
@@
 			)
 		)
-		(property "Codice" ""
+		(property "MPN" ""
 			(at 125.73 123.19 0)
 			(effects
@@
 			)
 		)
-		(property "Codice" "CRCW0805100RFKEA"
+		(property "MPN" "CRCW0805100RFKEA"
 			(at 142.24 133.35 90)
 			(effects
@@
 			)
 		)
-		(property "Codice" ""
+		(property "MPN" ""
 			(at 125.73 143.51 0)
 			(effects
@@
 			)
 		)
-		(property "Codice" "RMCF0805FT10K0"
+		(property "MPN" "RMCF0805FT10K0"
 			(at 172.72 45.72 90)
 			(effects
@@
 			)
 		)
-		(property "Codice" "RMCF0805FT10K0"
+		(property "MPN" "RMCF0805FT10K0"
 			(at 172.72 147.32 90)
 			(effects
@@
 			)
 		)
-		(property "Codice" "CRCW0805100RFKEA"
+		(property "MPN" "CRCW0805100RFKEA"
 			(at 142.24 52.07 90)
 			(effects
@@
 			)
 		)
-		(property "Codice" "RMCF0805FT10K0"
+		(property "MPN" "RMCF0805FT10K0"
 			(at 172.72 116.84 90)
 			(effects
@@
 			)
 		)
-		(property "Codice" ""
+		(property "MPN" ""
 			(at 125.73 82.55 0)
 			(effects
@@
 			)
 		)
-		(property "Codice" "RMCF0805FT10K0"
+		(property "MPN" "RMCF0805FT10K0"
 			(at 172.72 86.36 90)
 			(effects
@@
 			)
 		)
-		(property "Codice" "CRCW0805100RFKEA"
+		(property "MPN" "CRCW0805100RFKEA"
 			(at 142.24 102.87 90)
 			(effects
@@
 			)
 		)
-		(property "Codice" "RMCF0805FT10K0"
+		(property "MPN" "RMCF0805FT10K0"
 			(at 172.72 157.48 90)
 			(effects

Commit message: Rev B schematic: series termination, decoupling, assembly-ready parts
Function unchanged (no logic connection changes). Applied by
hardware/kicad/tile/scripts/revb_schematic.py:

- 33 ohm series resistors R201-R207 at every driver leaving the tile
  (L_clk, T_clk, L_latch, T_latch, B_data, R_data, B_W).
- 100 nF per logic IC (C201-C209); PWR_FLAGs on VCC, GND, VCC_T, GND_T.
- Values match the ordered parts (74LVC..., 74HC161); footprints:
  0603 passives, TI DCT land pattern for the 2G parts, standard
  SOT-23-5, SMD bulk capacitor, Kailh MX hot-swap sockets; Manufacturer
  and MPN fields, Link field dropped.
- Project footprint library with the hot-swap socket from
  keyswitch-kicad-library v2.3 (CC-BY-SA 4.0 with design exception).

Verified: netlist identical to rev A after collapsing R201-R207 and
ignoring C201-C209; ERC 0 errors (was 4).
Parts:
- R110, R111, R112, R113, R114, R115, R116, R117, R118, R119, R120, R121: value 100R -> 100; footprint Resistor_SMD:R_0805_2012Metric_Pad1.20x1.40mm_HandSolder -> Resistor_SMD:R_0603_1608Metric; Link https://www.digikey.it/it/products/detail/vishay-dale/CRCW0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 -> (none); MPN CRCW0805100RFKEA -> RC0603FR-07100RL; Manufacturer (none) -> Yageo
- R122, R123, R124, R125, R126, R127, R128, R129, R130, R131, R132, R133: footprint Resistor_SMD:R_0805_2012Metric_Pad1.20x1.40mm_HandSolder -> Resistor_SMD:R_0603_1608Metric; Link https://www.digikey.it/it/products/detail/stackpole-electro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 -> (none); MPN RMCF0805FT10K0 -> RC0603FR-0710KL; Manufacturer (none) -> Yageo
- SW101, SW102, SW103, SW104, SW105, SW106, SW107, SW108, SW109, SW110, SW111, SW112: footprint Button_Switch_Keyboard:SW_Cherry_MX_1.00u_PCB -> Switch_Keyboard_Hotswap_Kailh:SW_Hotswap_Kailh_MX_1.00u; MPN (none) -> CPG151101S11; Manufacturer (none) -> Kailh

Commit message: Rev B PCB: 4 layers, single-sided assembly, hot-swap sockets
Produced by hardware/kicad/tile/scripts/revb_pcb.py and
revb_pipeline.sh (rev-A board -> netlist update -> placement ->
Freerouting -> stitching/pours), fully reproducible.

- 4-layer 1.6 mm stack-up, In1 GND/GND_T and In2 VCC/VCC_T planes,
  Interboard net class 0.3 mm (~55 ohm), 4 mm ground stitching grid.
- Key board: Kailh MX hot-swap sockets and all resistors on B.Cu;
  switch centres unchanged (edge-trimmed socket footprint variant for
  the switches next to the stepped outline).
- Logic board: every SMD part on F.Cu; series resistors within 2.6 mm
  of their drivers; one 100 nF next to each IC.
- Fiducials (3 per board), board-only mouse bites, silkscreen revision
  v0.2, J107 courtyard margin reduced towards the SW111 socket.

Verified: DRC 0 errors, 0 unconnected, 0 schematic-parity issues;
switch/connector/outline invariants OK; SPICE tile hop as routed:
1 % overshoot (rev A: 22 %).
Parts:
- SW101, SW102, SW103, SW104, SW105, SW106, SW107, SW108, SW109, SW110, SW111, SW112: footprint Switch_Keyboard_Hotswap_Kailh:SW_Hotswap_Kailh_MX_1.00u -> Switch_Keyboard_Hotswap_Kailh:SW_Hotswap_Kailh_MX_1.00u_EdgeTrim
Changed lines of the file:
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@@
 			)
 		)
-		(property "Footprint" "Switch_Keyboard_Hotswap_Kailh:SW_Hotswap_Kailh_MX_1.00u"
+		(property "Footprint" "Switch_Keyboard_Hotswap_Kailh:SW_Hotswap_Kailh_MX_1.00u_EdgeTrim"
 			(at 125.73 67.31 0)
 			(hide yes)
@@
 			)
 		)
-		(property "Footprint" "Switch_Keyboard_Hotswap_Kailh:SW_Hotswap_Kailh_MX_1.00u"
+		(property "Footprint" "Switch_Keyboard_Hotswap_Kailh:SW_Hotswap_Kailh_MX_1.00u_EdgeTrim"
 			(at 125.73 57.15 0)
 			(hide yes)
@@
 			)
 		)
-		(property "Footprint" "Switch_Keyboard_Hotswap_Kailh:SW_Hotswap_Kailh_MX_1.00u"
+		(property "Footprint" "Switch_Keyboard_Hotswap_Kailh:SW_Hotswap_Kailh_MX_1.00u_EdgeTrim"
 			(at 125.73 107.95 0)
 			(hide yes)
@@
 			)
 		)
-		(property "Footprint" "Switch_Keyboard_Hotswap_Kailh:SW_Hotswap_Kailh_MX_1.00u"
+		(property "Footprint" "Switch_Keyboard_Hotswap_Kailh:SW_Hotswap_Kailh_MX_1.00u_EdgeTrim"
 			(at 125.73 128.27 0)
 			(hide yes)
@@
 			)
 		)
-		(property "Footprint" "Switch_Keyboard_Hotswap_Kailh:SW_Hotswap_Kailh_MX_1.00u"
+		(property "Footprint" "Switch_Keyboard_Hotswap_Kailh:SW_Hotswap_Kailh_MX_1.00u_EdgeTrim"
 			(at 125.73 46.99 0)
 			(hide yes)
@@
 			)
 		)
-		(property "Footprint" "Switch_Keyboard_Hotswap_Kailh:SW_Hotswap_Kailh_MX_1.00u"
+		(property "Footprint" "Switch_Keyboard_Hotswap_Kailh:SW_Hotswap_Kailh_MX_1.00u_EdgeTrim"
 			(at 125.73 97.79 0)
 			(hide yes)
@@
 			)
 		)
-		(property "Footprint" "Switch_Keyboard_Hotswap_Kailh:SW_Hotswap_Kailh_MX_1.00u"
+		(property "Footprint" "Switch_Keyboard_Hotswap_Kailh:SW_Hotswap_Kailh_MX_1.00u_EdgeTrim"
 			(at 125.73 148.59 0)
 			(hide yes)
@@
 			)
 		)
-		(property "Footprint" "Switch_Keyboard_Hotswap_Kailh:SW_Hotswap_Kailh_MX_1.00u"
+		(property "Footprint" "Switch_Keyboard_Hotswap_Kailh:SW_Hotswap_Kailh_MX_1.00u_EdgeTrim"
 			(at 125.73 36.83 0)
 			(hide yes)
@@
 			)
 		)
-		(property "Footprint" "Switch_Keyboard_Hotswap_Kailh:SW_Hotswap_Kailh_MX_1.00u"
+		(property "Footprint" "Switch_Keyboard_Hotswap_Kailh:SW_Hotswap_Kailh_MX_1.00u_EdgeTrim"
 			(at 125.73 87.63 0)
 			(hide yes)
@@
 			)
 		)
-		(property "Footprint" "Switch_Keyboard_Hotswap_Kailh:SW_Hotswap_Kailh_MX_1.00u"
+		(property "Footprint" "Switch_Keyboard_Hotswap_Kailh:SW_Hotswap_Kailh_MX_1.00u_EdgeTrim"
 			(at 125.73 118.11 0)
 			(hide yes)
@@
 			)
 		)
-		(property "Footprint" "Switch_Keyboard_Hotswap_Kailh:SW_Hotswap_Kailh_MX_1.00u"
+		(property "Footprint" "Switch_Keyboard_Hotswap_Kailh:SW_Hotswap_Kailh_MX_1.00u_EdgeTrim"
 			(at 125.73 138.43 0)
 			(hide yes)
@@
 			)
 		)
-		(property "Footprint" "Switch_Keyboard_Hotswap_Kailh:SW_Hotswap_Kailh_MX_1.00u"
+		(property "Footprint" "Switch_Keyboard_Hotswap_Kailh:SW_Hotswap_Kailh_MX_1.00u_EdgeTrim"
 			(at 125.73 77.47 0)
 			(hide yes)
