File: hardware/kicad/revc-mcu-tile/revc_mcu.kicad_pcb (KiCad board)
At the start: 2 copper layers, 90.8 x 46.7 mm, 40 parts, among them SW101 SW_Push, SW102 SW_Push, SW103 SW_Push, SW104 SW_Push, SW105 SW_Push, SW106 SW_Push, SW107 SW_Push, SW108 SW_Push, SW109 SW_Push, SW110 SW_Push, SW111 SW_Push, SW112 SW_Push, U1 ATtiny1616-MNR

Commit message: Rev C MCU tile: KiCad schematic drives the board
- revc_mcu_circuit.py defines the circuit once; revc_mcu_schematic.py
  writes it as a KiCad schematic (stock symbols embedded, stable UUIDs).
- The board build takes every net, value and field from the netlist that
  kicad-cli exports, checks that board and schematic hold the same parts
  and footprints, and links footprints to symbols.
- Pin swapping: the 15 interchangeable MCU signals get the pins in the
  angular order of their destinations; stored in pinmap.json (also for
  the firmware), and the schematic is redrawn when it changes.
- LED chain starts at D6, next to the MCU; the flow tries MCU
  orientations until the board is clean.
- Flow: ERC, then DRC with schematic parity. Result kept in
  hardware/kicad/revc-mcu-tile/ as a normal KiCad project: ERC clean,
  DRC 0 errors, 0 unconnected, 0 parity issues, no via-in-pad.
Parts:
- removed C10, C12, C13, C14, C15: 100n, Capacitor_SMD:C_0603_1608Metric
- removed C11: 4u7, Capacitor_SMD:C_0805_2012Metric
- added C5: 100n, Capacitor_SMD:C_0603_1608Metric, B.Cu at (112.8, 90.0)
- added C6: 100n, Capacitor_SMD:C_0603_1608Metric, B.Cu at (167.9, 90.0)
- added J1: spring contacts right, revc:EdgeContacts_right, B.Cu at (189.1, 69.5)
- added J2: edge pads left, revc:EdgeContacts_left, B.Cu at (118.5, 69.5)
- added J3: spring contacts bottom, revc:EdgeContacts_bottom, B.Cu at (145.6, 91.0)
- added J4: edge pads top, revc:EdgeContacts_top, B.Cu at (154.7, 45.9)
- C1: value contacts right -> 100n; footprint revc:EdgeContacts_right -> Capacitor_SMD:C_0603_1608Metric
- C2: value contacts left -> 4u7; footprint revc:EdgeContacts_left -> Capacitor_SMD:C_0805_2012Metric
- C3: value contacts bottom -> 100n; footprint revc:EdgeContacts_bottom -> Capacitor_SMD:C_0603_1608Metric
- C4: value contacts top -> 100n; footprint revc:EdgeContacts_top -> Capacitor_SMD:C_0603_1608Metric
- SW1: renamed from SW102; value SW_Push -> MX hot-swap
- SW10: renamed from SW105; value SW_Push -> MX hot-swap
- SW11: renamed from SW112; value SW_Push -> MX hot-swap
- SW12: renamed from SW111; value SW_Push -> MX hot-swap
- SW2: renamed from SW101; value SW_Push -> MX hot-swap
- SW3: renamed from SW108; value SW_Push -> MX hot-swap
- SW4: renamed from SW107; value SW_Push -> MX hot-swap
- SW5: renamed from SW104; value SW_Push -> MX hot-swap
- SW6: renamed from SW103; value SW_Push -> MX hot-swap
- SW7: renamed from SW110; value SW_Push -> MX hot-swap
- SW8: renamed from SW109; value SW_Push -> MX hot-swap
- SW9: renamed from SW106; value SW_Push -> MX hot-swap
- moved C2 36.6 mm to (154.3, 61.7)
- moved C1 35.3 mm to (154.3, 64.0)
- moved C4 34.6 mm to (186.2, 60.2), turned to 90 degrees
- moved C3 31.3 mm to (135.9, 61.2)
- turned D10 to 180 degrees
- turned D11 to 180 degrees
- turned D12 to 180 degrees
- turned D4 to 180 degrees
- turned D5 to 0 degrees
- turned D7 to 0 degrees
- turned D9 to 180 degrees
- turned U1 to 90 degrees
Connections:
- C1 pad 2: DATA_R -> GND
- C2 pad 2: DATA_L -> GND
- C3 pad 2: DATA_B -> GND
- C4 pad 2: DATA_T -> GND
- D1 pad 2: LED_DIN -> LED_D5
- D10 pad 2: LED_D9 -> LED_D11
- D11 pad 2: LED_D10 -> LED_D12
- D12 pad 2: LED_D11 -> LED_D7
- D12 pad 4: LED_END -> LED_D12
- D6 pad 2: LED_D7 -> LED_DIN
- D9 pad 2: LED_D5 -> LED_D10
- D9 pad 4: LED_D9 -> unconnected-(D9-DOUT-Pad4)
- U1 pad 1: K1 -> K12
- U1 pad 10: K10 -> K1
- U1 pad 11: K9 -> K6
- U1 pad 13: K8 -> K2
- U1 pad 14: K7 -> DATA_T_MCU
- U1 pad 15: DATA_T_MCU -> K3
- U1 pad 16: DATA_L_MCU -> K4
- U1 pad 17: LED_DIN -> K7
- U1 pad 18: K12 -> K8
- U1 pad 2: K2 -> K11
- U1 pad 5: K3 -> K10
- U1 pad 6: K4 -> LED_DIN
- U1 pad 7: K5 -> K9
- U1 pad 8: K6 -> DATA_L_MCU
- U1 pad 9: K11 -> K5
Routing:
- net LED_D3: track 13.5 -> 40.9 mm
- net LED_DIN: track 32.3 -> 6.04 mm, vias 2 -> 0
- net K11: track 35.5 -> 10.4 mm, vias 2 -> 0
- net DATA_R_MCU: track 55.6 -> 33.3 mm, vias 6 -> 0
- net GND: track 193.2 -> 175.5 mm, vias 118 -> 128
- net LED_D9: track 14.4 -> 0.00 mm
- net LED_D12: track 0.00 -> 14.1 mm
- net K9: track 47.2 -> 33.8 mm, vias 2 -> 0
- net K1: track 37.7 -> 26.1 mm
- net K4: track 73.3 -> 62.3 mm
- net K12: track 36.9 -> 27.1 mm, vias 2 -> 0
- net LED_D6: track 13.5 -> 21.1 mm, vias 0 -> 2
- net K2: track 36.4 -> 29.1 mm
- net LED_D8: track 13.5 -> 20.3 mm, vias 0 -> 2
- net DATA_B_MCU: track 28.0 -> 34.6 mm
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