File: hardware/experiments/simple-tile/fpga/board/out/kicad/tile_gw1nz.kicad_pcb (KiCad board)
At the start: 2 copper layers, 90.8 x 46.7 mm, 58 parts, among them SW1 Kailh MX hotswap, SW10 Kailh MX hotswap, SW11 Kailh MX hotswap, SW12 Kailh MX hotswap, SW2 Kailh MX hotswap, SW3 Kailh MX hotswap, SW4 Kailh MX hotswap, SW5 Kailh MX hotswap, SW6 Kailh MX hotswap, SW7 Kailh MX hotswap, SW8 Kailh MX hotswap, SW9 Kailh MX hotswap, U1 GW1NZ-LV1QN48C6/I5, U2 LDO-1V2

Commit message: Checkpoint FPGA electrical design and incomplete four-layer routing trial
Work stopped 2026-10-16 15:18 CEST by user request. Four-layer GW1NZ
ground-pour repair left at: 0 error-severity DRC, 150 warnings, 54 ground
opens, 44/52 post-import power attaches, 2 copper-neck warnings open,
8 unplaced. No acceptance gate closed.
Parts:
- added C8: 1u, C8, B.Cu at (-8.77, 19.2)
- added C9: 1u, C9, B.Cu at (-12.3, 21.4)
- added R10: 0R, R10, B.Cu at (-0.09, 5.85)
- added R11: 0R, R11, B.Cu at (0.91, 10.8)
- added R7: 0R, R7, B.Cu at (-0.09, 3.10)
- added R8: 0R, R8, B.Cu at (12.4, 14.1)
- added R9: 0R, R9, B.Cu at (-0.09, 4.45)
- U2: value LDO-1V2 -> TLV75512PDBVR
- moved TP_JTAGSEL 23.3 mm to (-2.39, 3.15)
- moved TP_VCC1V2 20.4 mm to (-2.39, 5.40)
- moved TP_TDO 19.1 mm to (17.4, 7.40)
- moved TP_DONE 18.8 mm to (17.6, 9.65)
- moved TP_READY 18.6 mm to (17.6, 15.2)
- moved TP_TMS 10.3 mm to (-0.64, 13.9)
- moved TP_RECFG 4.51 mm to (17.6, 11.9)
- moved TP_TDI 2.02 mm to (-1.14, 7.65)
- moved TP_VCC 0.56 mm to (-6.01, 18.7)
Connections:
- U1 pad 19: L_clk -> L_clk_DRV
- U1 pad 27: B_W -> B_W_DRV
- U1 pad 30: B_data -> B_data_DRV
- U1 pad 31: L_latch -> L_latch_DRV
- U1 pad 35: T_clk -> T_clk_DRV
