File: hardware/experiments/simple-tile/fpga/board/out/kicad/tile_up5k.kicad_pcb (KiCad board)
At the start: 2 copper layers, 90.8 x 46.7 mm, 70 parts, among them SW1 Kailh MX hotswap, SW10 Kailh MX hotswap, SW11 Kailh MX hotswap, SW12 Kailh MX hotswap, SW2 Kailh MX hotswap, SW3 Kailh MX hotswap, SW4 Kailh MX hotswap, SW5 Kailh MX hotswap, SW6 Kailh MX hotswap, SW7 Kailh MX hotswap, SW8 Kailh MX hotswap, SW9 Kailh MX hotswap, U2 LDO-1V2, U3 SPI-FLASH

Commit message: Checkpoint FPGA electrical design and incomplete four-layer routing trial
Work stopped 2026-10-16 15:18 CEST by user request. Four-layer GW1NZ
ground-pour repair left at: 0 error-severity DRC, 150 warnings, 54 ground
opens, 44/52 post-import power attaches, 2 copper-neck warnings open,
8 unplaced. No acceptance gate closed.
Parts:
- added C11: 1u, C11, B.Cu at (-11.5, 19.2)
- added C12: 1u, C12, B.Cu at (-8.27, 19.2)
- U2: value LDO-1V2 -> TLV75512PDBVR
- moved TP_VCC 5.85 mm to (-9.77, 24.4)
Changed lines of the file:
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@@
 		)
 	)
-	(property "Value" "LDO-1V2"
+	(property "Value" "TLV75512PDBVR"
 		(at 0 2.4 0)
 		(layer "B.Fab")
@@
 	)
 )
+(footprint "C11"
+	(version 20260206)
+	(generator "kicad-footprint-generator")
+	(layer "B.Cu")
+	(at -11.5150 19.2000 0)
+	(descr "Capacitor SMD 0603 (1608 Metric), square (rectangular) end terminal, IPC-7351 nominal, (Body size source: IPC-SM-782 page 76, https://www.pcb-3d.com/wordpress/wp-content/uploads/ipc-sm-782a_amendment_1_and_2.pdf)")
+	(tags "capacitor")
+	(property "Reference" "C11"
+		(at 0 -1.43 0)
+		(layer "B.SilkS")
+		(effects (justify mirror)
+			(font
+				(size 1 1)
+				(thickness 0.15)
+			)
+		)
+	)
+	(property "Value" "1u"
+		(at 0 1.43 0)
+		(layer "B.Fab")
+		(effects (justify mirror)
+			(font
+				(size 1 1)
+				(thickness 0.15)
+			)
+		)
+	)
+	(property "KiLib_Generator" "SMD_2terminal_chip_molded"
+		(at 0 0 0)
+		(layer "B.SilkS")
+		(hide yes)
+		(effects (justify mirror)
+			(font
+				(size 1 1)
+				(thickness 0.15)
+			)
+		)
+	)
+	(attr smd)
+	(duplicate_pad_numbers_are_jumpers no)
+	(fp_line
+		(start 0.14058 -0.51)
+		(end -0.14058 -0.51)
+		(stroke
+			(width 0.12)
+			(type solid)
+		)
+		(layer "B.SilkS")
+	)
+	(fp_line
+		(start 0.14058 0.51)
+		(end -0.14058 0.51)
+		(stroke
+			(width 0.12)
+			(type solid)
+		)
+		(layer "B.SilkS")
+	)
+	(fp_rect
+		(start -1.48 -0.73) (end 1.48 0.73)
+		(stroke
+			(width 0.05)
+			(type solid)
+		)
+		(fill no)
+		(layer "B.CrtYd")
+	)
+	(fp_rect
+		(start -0.8 -0.4) (end 0.8 0.4)
+		(stroke
+			(width 0.1)
+			(type solid)
+		)
+		(fill no)
+		(layer "B.Fab")
+	)
+	(fp_text user "${REFERENCE}"
+		(at 0 0 0)
+		(layer "B.Fab")
+		(effects (justify mirror)
+			(font
+				(size 0.4 0.4)
+				(thickness 0.06)
+			)
+		)
+	)
+	(pad "1" smd roundrect
+		(at 0.775 0)
+		(size 0.9 0.95)
+		(layers "B.Cu" "B.Mask" "B.Paste")
+		(roundrect_rratio 0.25)
+	 (net 1 "VCC"))
+	(pad "2" smd roundrect
+		(at -0.775 0)
+		(size 0.9 0.95)
+		(layers "B.Cu" "B.Mask" "B.Paste")
+		(roundrect_rratio 0.25)
+	 (net 14 "GND"))
+	(embedded_fonts no)
+	(model "${KICAD10_3DMODEL_DIR}/Capacitor_SMD.3dshapes/C_0603_1608Metric.step"
+		(offset
+			(xyz 0 0 0)
+		)
+		(scale
+			(xyz 1 1 1)
+		)
+		(rotate
+			(xyz 0 0 0)
+		)
+	)
+)
+(footprint "C12"
+	(version 20260206)
+	(generator "kicad-footprint-generator")
+	(layer "B.Cu")
+	(at -8.2650 19.2000 0)
+	(descr "Capacitor SMD 0603 (1608 Metric), square (rectangular) end terminal, IPC-7351 nominal, (Body size source: IPC-SM-782 page 76, https://www.pcb-3d.com/wordpress/wp-content/uploads/ipc-sm-782a_amendment_1_and_2.pdf)")
+	(tags "capacitor")
+	(property "Reference" "C12"
+		(at 0 -1.43 0)
+		(layer "B.SilkS")
+		(effects (justify mirror)
+			(font
+				(size 1 1)
+				(thickness 0.15)
+			)
+		)
+	)
+	(property "Value" "1u"
+		(at 0 1.43 0)
+		(layer "B.Fab")
+		(effects (justify mirror)
+			(font
+				(size 1 1)
+				(thickness 0.15)
+			)
+		)
+	)
+	(property "KiLib_Generator" "SMD_2terminal_chip_molded"
+		(at 0 0 0)
+		(layer "B.SilkS")
+		(hide yes)
+		(effects (justify mirror)
+			(font
+				(size 1 1)
+				(thickness 0.15)
+			)
+		)
+	)
+	(attr smd)
+	(duplicate_pad_numbers_are_jumpers no)
+	(fp_line
+		(start 0.14058 -0.51)
+		(end -0.14058 -0.51)
+		(stroke
+			(width 0.12)
+			(type solid)
+		)
+		(layer "B.SilkS")
+	)
+	(fp_line
+		(start 0.14058 0.51)
+		(end -0.14058 0.51)
+		(stroke
+			(width 0.12)
+			(type solid)
+		)
+		(layer "B.SilkS")
+	)
+	(fp_rect
+		(start -1.48 -0.73) (end 1.48 0.73)
+		(stroke
+			(width 0.05)
+			(type solid)
+		)
+		(fill no)
+		(layer "B.CrtYd")
+	)
+	(fp_rect
+		(start -0.8 -0.4) (end 0.8 0.4)
+		(stroke
+			(width 0.1)
+			(type solid)
+		)
+		(fill no)
+		(layer "B.Fab")
+	)
+	(fp_text user "${REFERENCE}"
+		(at 0 0 0)
+		(layer "B.Fab")
+		(effects (justify mirror)
+			(font
+				(size 0.4 0.4)
+				(thickness 0.06)
+			)
+		)
+	)
+	(pad "1" smd roundrect
+		(at 0.775 0)
+		(size 0.9 0.95)
+		(layers "B.Cu" "B.Mask" "B.Paste")
+		(roundrect_rratio 0.25)
+	 (net 29 "VCC1V2"))
+	(pad "2" smd roundrect
+		(at -0.775 0)
+		(size 0.9 0.95)
+		(layers "B.Cu" "B.Mask" "B.Paste")
+		(roundrect_rratio 0.25)
+	 (net 14 "GND"))
+	(embedded_fonts no)
+	(model "${KICAD10_3DMODEL_DIR}/Capacitor_SMD.3dshapes/C_0603_1608Metric.step"
+		(offset
+			(xyz 0 0 0)
+		)
+		(scale
+			(xyz 1 1 1)
+		)
+		(rotate
+			(xyz 0 0 0)
+		)
+	)
+)
 (footprint "R10"
 	(version 20260206)
@@
 	(generator_version "10.0")
 	(layer "B.Cu")
-	(at -11.7650 18.9500 0)
+	(at -9.7650 24.4500 0)
 	(descr "SMD pad as test Point, diameter 1.0mm")
 	(tags "test point SMD pad")
